File: MGB-xCPU/audio.sch (KiCad schematic (older format))
At the start: 39 parts, among them P5 Headphones, U3 IR3R53N

Commit message: Update libraries and regenerate schematics
Parts:
- C31: symbol Device:CP -> Device:C_Polarized
- EM1, EM2, EM3: symbol Device:Ferrite_Bead_Small -> Device:FerriteBead_Small
Changed lines of the file:
@@
 Title "MGB-xCPU - Analog audio"
 Date "2020-09-19"
-Rev "A"
+Rev "B"
 Comp "https://gekkio.fi"
 Comment1 "https://github.com/gekkio/gb-schematics"
@@
 $EndComp
 $Comp
-L Device:CP C31
+L Device:C_Polarized C31
 U 1 1 5F65F2ED
 P 9000 5100
+AR Path="/5F65F2ED" Ref="C31"  Part="1"
+AR Path="/5F624AB5/5F65F2ED" Ref="C31"  Part="1"
 F 0 "C31" H 9118 5146 50  0000 L CNN
 F 1 "100uF" H 9118 5055 50  0000 L CNN
@@
 $EndComp
 $Comp
-L Device:Ferrite_Bead_Small EM?
+L Device:FerriteBead_Small EM?
 U 1 1 5F65F317
 P 9150 3500
@@
 $EndComp
 $Comp
-L Device:Ferrite_Bead_Small EM?
+L Device:FerriteBead_Small EM?
 U 1 1 5F65F329
 P 9150 2250
@@
 	10050 3600 9850 3600
 $Comp
-L Device:Ferrite_Bead_Small EM?
+L Device:FerriteBead_Small EM?
 U 1 1 5F65F331
 P 9150 2450
