File: MGB-xCPU/lcd.sch (KiCad schematic (older format))
At the start: 42 parts, among them P2 LCD FPC, Q1 2SA1576A, U4 IR3E02

Commit message: Update libraries and regenerate schematics
Parts:
- JP1, JP2, JP3, JP4, JP5, JP6, JP7, JP8, JP9: value Jumper_NC_Small -> SolderJumper_2_Bridged; symbol Device:Jumper_NC_Small -> Jumper:SolderJumper_2_Bridged
Other:
- moved on the sheet: C20, C21, C22, C23, C24, C28, C3, P2, Q1, R1, TP64, TP65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
