File: MGB-xCPU/power.sch (KiCad schematic (older format))
At the start: 29 parts, among them P4 DC 3V, Q2 2SC4081, SW1 SP3T, U5 DC/DC

Commit message: Update libraries and regenerate schematics
Parts:
- C29, C30, C32: symbol Device:CP -> Device:C_Polarized
Changed lines of the file:
@@
 Title "MGB-xCPU - Power"
 Date "2020-09-19"
-Rev "A"
+Rev "B"
 Comp "https://gekkio.fi"
 Comment1 "https://github.com/gekkio/gb-schematics"
@@
 $EndComp
 $Comp
-L Device:CP C?
+L Device:C_Polarized C?
 U 1 1 5ED09B7B
 P 3200 4000
@@
 Connection ~ 3200 3750
 $Comp
-L Device:CP C?
+L Device:C_Polarized C?
 U 1 1 5ED09B9F
 P 3200 4500
@@
 $EndComp
 $Comp
-L Device:CP C?
+L Device:C_Polarized C?
 U 1 1 5ED09BAC
 P 2050 4000
