File: MGB-xCPU/MGB-xCPU.kicad_sch (KiCad schematic)
At the start: 56 parts, among them P1 GameBoy_Cartridge, U1 CPU MGB, U2 LH52A64N, U6 PST9135N, X1 4.194304 MHz

Commit message: Release: MGB-xCPU rev D
Parts:
- added CL1, CL2, CL3, CL4, CL5: TestPoint, symbol Connector:TestPoint
Connections:
- net A14: now also CL5.1
- net GND: now also CL3.1, CL4.1
- net VDD: now also CL1.1, CL2.1
Other:
- moved on the sheet: U2

Commit message: Remove Farad/Henry units
Parts:
- C1, C2: value 25pF -> 25p
- C10, C11, C12: value 10nF -> 10n
- C17: value 100nF -> 100n
Changed lines of the file:
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@@
       (effects (font (size 1.27 1.27)) (justify left))
     )
-    (property "Value" "10nF" (at 272.161 154.813 0)
+    (property "Value" "10n" (at 272.161 154.813 0)
       (effects (font (size 1.27 1.27)) (justify left))
     )
@@
       (effects (font (size 1.27 1.27)) (justify left))
     )
-    (property "Value" "10nF" (at 230.251 154.813 0)
+    (property "Value" "10n" (at 230.251 154.813 0)
       (effects (font (size 1.27 1.27)) (justify left))
     )
@@
       (effects (font (size 1.27 1.27)) (justify left))
     )
-    (property "Value" "25pF" (at 28.321 114.173 0)
+    (property "Value" "25p" (at 28.321 114.173 0)
       (effects (font (size 1.27 1.27)) (justify left))
     )
@@
       (effects (font (size 1.27 1.27)) (justify left))
     )
-    (property "Value" "25pF" (at 41.021 114.173 0)
+    (property "Value" "25p" (at 41.021 114.173 0)
       (effects (font (size 1.27 1.27)) (justify left))
     )
@@
       (effects (font (size 1.27 1.27)) (justify left))
     )
-    (property "Value" "100nF" (at 43.561 69.723 0)
+    (property "Value" "100n" (at 43.561 69.723 0)
       (effects (font (size 1.27 1.27)) (justify left))
     )
@@
       (effects (font (size 1.27 1.27)) (justify left))
     )
-    (property "Value" "10nF" (at 112.141 167.513 0)
-      (effects (font (size 1.27 1.27)) (justify left))
-    )
+    (property "Value" "10n" (at 112.141 167.513 0)
+      (effects (font (size 1.27 1.27)) (justify left))
+    )
