File: MGB-xCPU/power.kicad_sch (KiCad schematic)
At the start: 29 parts, among them P4 DC 3V, Q2 2SC4081, SW1 SP3T, U5 DC/DC

Commit message: Add electrolytic capacitor ratings
Parts:
- C29: Rating (none) -> 25V
- C30, C32: Rating (none) -> 6.3V
Other:
- moved on the sheet: C33
Changed lines of the file:
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@@
-    (stroke (width 0) (type default) (color 0 0 0 0))
-  )
-  (wire (pts (xy 92.71 105.41) (xy 92.71 107.95))
     (stroke (width 0) (type default) (color 0 0 0 0))
   )
@@
     (stroke (width 0) (type default) (color 0 0 0 0))
   )
+  (wire (pts (xy 95.25 95.25) (xy 95.25 97.79))
+    (stroke (width 0) (type default) (color 0 0 0 0))
+  )
+  (wire (pts (xy 95.25 107.95) (xy 95.25 105.41))
+    (stroke (width 0) (type default) (color 0 0 0 0))
+  )
   (wire (pts (xy 69.85 67.31) (xy 105.41 67.31))
     (stroke (width 0) (type default) (color 0 0 0 0))
@@
     (stroke (width 0) (type default) (color 0 0 0 0))
   )
-  (wire (pts (xy 92.71 95.25) (xy 92.71 97.79))
-    (stroke (width 0) (type default) (color 0 0 0 0))
-  )
   (wire (pts (xy 60.96 64.77) (xy 60.96 67.31))
     (stroke (width 0) (type default) (color 0 0 0 0))
@@
     (stroke (width 0) (type default) (color 0 0 0 0))
   )
-  (wire (pts (xy 81.28 95.25) (xy 92.71 95.25))
+  (wire (pts (xy 81.28 95.25) (xy 95.25 95.25))
     (stroke (width 0) (type default) (color 0 0 0 0))
   )
@@
     (stroke (width 0) (type default) (color 0 0 0 0))
   )
-  (wire (pts (xy 92.71 107.95) (xy 81.28 107.95))
+  (wire (pts (xy 81.28 107.95) (xy 95.25 107.95))
     (stroke (width 0) (type default) (color 0 0 0 0))
   )
@@
   )
   (symbol (lib_id "Device:C_Polarized") (at 81.28 101.6 0) (unit 1)
-    (in_bom yes) (on_board yes)
-    (property "Reference" "C30" (id 0) (at 84.2772 100.4316 0)
-      (effects (font (size 1.27 1.27)) (justify left))
-    )
-    (property "Value" "330uF" (id 1) (at 84.2772 102.743 0)
+    (in_bom yes) (on_board yes) (fields_autoplaced)
+    (property "Reference" "C30" (id 0) (at 85.09 98.1709 0)
+      (effects (font (size 1.27 1.27)) (justify left))
+    )
+    (property "Value" "330uF" (id 1) (at 85.09 100.7109 0)
       (effects (font (size 1.27 1.27)) (justify left))
     )
@@
     (property "Datasheet" "~" (id 3) (at 81.28 101.6 0)
       (effects (font (size 1.27 1.27)) hide)
+    )
+    (property "Rating" "6.3V" (id 4) (at 85.09 103.2509 0)
+      (effects (font (size 1.27 1.27)) (justify left))
     )
     (pin "1")
@@
     (pin "1")
   )
-  (symbol (lib_id "Device:C") (at 92.71 101.6 0) (unit 1)
+  (symbol (lib_id "Device:C") (at 95.25 101.6 0) (unit 1)
     (in_bom yes) (on_board yes)
-    (property "Reference" "C33" (id 0) (at 95.631 100.4316 0)
-      (effects (font (size 1.27 1.27)) (justify left))
-    )
-    (property "Value" "6.8uF" (id 1) (at 95.631 102.743 0)
-      (effects (font (size 1.27 1.27)) (justify left))
-    )
-    (property "Footprint" "" (id 2) (at 93.6752 105.41 0)
-      (effects (font (size 1.27 1.27)) hide)
-    )
-    (property "Datasheet" "~" (id 3) (at 92.71 101.6 0)
+    (property "Reference" "C33" (id 0) (at 98.171 100.4316 0)
+      (effects (font (size 1.27 1.27)) (justify left))
+    )
+    (property "Value" "6.8uF" (id 1) (at 98.171 102.743 0)
+      (effects (font (size 1.27 1.27)) (justify left))
+    )
+    (property "Footprint" "" (id 2) (at 96.2152 105.41 0)
+      (effects (font (size 1.27 1.27)) hide)
+    )
+    (property "Datasheet" "~" (id 3) (at 95.25 101.6 0)
       (effects (font (size 1.27 1.27)) hide)
     )
@@
   )
   (symbol (lib_id "Device:C_Polarized") (at 81.28 114.3 0) (mirror y) (unit 1)
-    (in_bom yes) (on_board yes)
-    (property "Reference" "C29" (id 0) (at 84.2772 113.1316 0)
-      (effects (font (size 1.27 1.27)) (justify right))
-    )
-    (property "Value" "33uF" (id 1) (at 84.2772 115.443 0)
+    (in_bom yes) (on_board yes) (fields_autoplaced)
+    (property "Reference" "C29" (id 0) (at 85.09 110.8709 0)
+      (effects (font (size 1.27 1.27)) (justify right))
+    )
+    (property "Value" "33uF" (id 1) (at 85.09 113.4109 0)
       (effects (font (size 1.27 1.27)) (justify right))
     )
@@
       (effects (font (size 1.27 1.27)) hide)
     )
+    (property "Rating" "25V" (id 4) (at 85.09 115.9509 0)
+      (effects (font (size 1.27 1.27)) (justify right))
+    )
     (pin "1")
     (pin "2")
   )
   (symbol (lib_id "Device:C_Polarized") (at 52.07 101.6 0) (unit 1)
-    (in_bom yes) (on_board yes)
-    (property "Reference" "C32" (id 0) (at 49.0982 100.4316 0)
-      (effects (font (size 1.27 1.27)) (justify right))
-    )
-    (property "Value" "100uF" (id 1) (at 49.0982 102.743 0)
+    (in_bom yes) (on_board yes) (fields_autoplaced)
+    (property "Reference" "C32" (id 0) (at 48.26 98.1709 0)
+      (effects (font (size 1.27 1.27)) (justify right))
+    )
+    (property "Value" "100uF" (id 1) (at 48.26 100.7109 0)
       (effects (font (size 1.27 1.27)) (justify right))
     )
@@
       (effects (font (size 1.27 1.27)) hide)
     )
-    (pin "1")
+    (property "Rating" "6.3V" (id 4) (at 48.26 103.2509 0)
+      (effects (font (size 1.27 1.27)) (justify right))
+    )
+    (pin "1")

Commit message: Add missing C35 value
Raw measurements:
- 0603 imperial
- 101.4 pF @ 1kHz
Parts:
- C35: value C -> 100pF
Other:
- moved on the sheet: C35
Changed lines of the file:
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@@
   (junction (at 85.09 52.07) (diameter 0) (color 0 0 0 0)
   )
-  (junction (at 74.93 52.07) (diameter 0) (color 0 0 0 0)
+  (junction (at 72.39 52.07) (diameter 0) (color 0 0 0 0)
   )
   (junction (at 97.79 52.07) (diameter 0) (color 0 0 0 0)
@@
     (stroke (width 0) (type default) (color 0 0 0 0))
   )
-  (wire (pts (xy 74.93 52.07) (xy 85.09 52.07))
+  (wire (pts (xy 72.39 52.07) (xy 85.09 52.07))
     (stroke (width 0) (type default) (color 0 0 0 0))
   )
@@
     (stroke (width 0) (type default) (color 0 0 0 0))
   )
-  (wire (pts (xy 74.93 52.07) (xy 74.93 54.61))
+  (wire (pts (xy 72.39 52.07) (xy 72.39 54.61))
     (stroke (width 0) (type default) (color 0 0 0 0))
   )
@@
     (stroke (width 0) (type default) (color 0 0 0 0))
   )
-  (wire (pts (xy 60.96 64.77) (xy 74.93 64.77))
+  (wire (pts (xy 60.96 64.77) (xy 72.39 64.77))
     (stroke (width 0) (type default) (color 0 0 0 0))
   )
@@
     (stroke (width 0) (type default) (color 0 0 0 0))
   )
-  (wire (pts (xy 58.42 52.07) (xy 74.93 52.07))
+  (wire (pts (xy 58.42 52.07) (xy 72.39 52.07))
     (stroke (width 0) (type default) (color 0 0 0 0))
   )
@@
     (stroke (width 0) (type default) (color 0 0 0 0))
   )
-  (wire (pts (xy 69.85 67.31) (xy 105.41 67.31))
+  (wire (pts (xy 67.31 67.31) (xy 105.41 67.31))
     (stroke (width 0) (type default) (color 0 0 0 0))
   )
@@
     (stroke (width 0) (type default) (color 0 0 0 0))
   )
-  (wire (pts (xy 69.85 54.61) (xy 69.85 67.31))
+  (wire (pts (xy 67.31 54.61) (xy 67.31 67.31))
     (stroke (width 0) (type default) (color 0 0 0 0))
   )
@@
     (stroke (width 0) (type default) (color 0 0 0 0))
   )
-  (wire (pts (xy 74.93 64.77) (xy 74.93 62.23))
-    (stroke (width 0) (type default) (color 0 0 0 0))
-  )
-  (wire (pts (xy 69.85 54.61) (xy 58.42 54.61))
+  (wire (pts (xy 72.39 64.77) (xy 72.39 62.23))
+    (stroke (width 0) (type default) (color 0 0 0 0))
+  )
+  (wire (pts (xy 67.31 54.61) (xy 58.42 54.61))
     (stroke (width 0) (type default) (color 0 0 0 0))
   )
@@
     (pin "1")
   )
-  (symbol (lib_id "Device:C") (at 74.93 58.42 0) (unit 1)
-    (in_bom yes) (on_board yes)
-    (property "Reference" "C35" (id 0) (at 77.851 57.2516 0)
-      (effects (font (size 1.27 1.27)) (justify left))
-    )
-    (property "Value" "C" (id 1) (at 77.851 59.563 0)
-      (effects (font (size 1.27 1.27)) (justify left))
-    )
-    (property "Footprint" "" (id 2) (at 75.8952 62.23 0)
-      (effects (font (size 1.27 1.27)) hide)
-    )
-    (property "Datasheet" "~" (id 3) (at 74.93 58.42 0)
-      (effects (font (size 1.27 1.27)) hide)
-    )
+  (symbol (lib_id "Device:C") (at 72.39 58.42 0) (unit 1)
+    (in_bom yes) (on_board yes)
+    (property "Reference" "C35" (id 0) (at 75.311 57.2516 0)
+      (effects (font (size 1.27 1.27)) (justify left))
+    )
+    (property "Value" "100pF" (id 1) (at 75.311 59.563 0)
+      (effects (font (size 1.27 1.27)) (justify left))
+    )
+    (property "Footprint" "" (id 2) (at 73.3552 62.23 0)
+      (effects (font (size 1.27 1.27)) hide)
+    )
+    (property "Datasheet" "~" (id 3) (at 72.39 58.42 0)
+      (effects (font (size 1.27 1.27)) hide)
+    )

Commit message: Release: MGB-xCPU rev C
Other:
- title: MGB-xCPU - Power -> MGB-xCPU
Changed lines of the file:
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@@
   (paper "A4")
   (title_block
-    (title "MGB-xCPU - Power")
-    (date "2020-09-19")
-    (rev "B")
+    (title "MGB-xCPU")
+    (date "2022-01-02")
+    (rev "C")
     (company "https://gekkio.fi")
     (comment 1 "https://github.com/gekkio/gb-schematics")

Commit message: Remove Farad/Henry units
Parts:
- C29: value 33uF -> 33u
- C30: value 330uF -> 330u
- C32: value 100uF -> 100u
- C33: value 6.8uF -> 6.8u
- C35: value 100pF -> 100p
Changed lines of the file:
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@@
       (effects (font (size 1.27 1.27)) (justify left))
     )
-    (property "Value" "330uF" (at 85.09 100.7109 0)
+    (property "Value" "330u" (at 85.09 100.7109 0)
       (effects (font (size 1.27 1.27)) (justify left))
     )
@@
       (effects (font (size 1.27 1.27)) (justify left))
     )
-    (property "Value" "6.8uF" (at 98.171 102.743 0)
+    (property "Value" "6.8u" (at 98.171 102.743 0)
       (effects (font (size 1.27 1.27)) (justify left))
     )
@@
       (effects (font (size 1.27 1.27)) (justify right))
     )
-    (property "Value" "33uF" (at 85.09 113.4109 0)
+    (property "Value" "33u" (at 85.09 113.4109 0)
       (effects (font (size 1.27 1.27)) (justify right))
     )
@@
       (effects (font (size 1.27 1.27)) (justify right))
     )
-    (property "Value" "100uF" (at 48.26 100.7109 0)
+    (property "Value" "100u" (at 48.26 100.7109 0)
       (effects (font (size 1.27 1.27)) (justify right))
     )
@@
       (effects (font (size 1.27 1.27)) (justify left))
     )
-    (property "Value" "100pF" (at 75.311 59.563 0)
-      (effects (font (size 1.27 1.27)) (justify left))
-    )
+    (property "Value" "100p" (at 75.311 59.563 0)
+      (effects (font (size 1.27 1.27)) (justify left))
+    )

Commit message: Add some power-related information
Parts:
- BT1: value Battery -> 2xAAA
Other:
- note added: "Main power inputs (DC jack, battery) 0.7W"
- note added: "Plug: 2.35 mm x 0.75 mm Center positive polarity"
- note removed: "Main power inputs (DC jack, battery)"
Changed lines of the file:
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@@
     (effects (font (size 1.27 1.27)) (justify left bottom))
+  )
+  (text "Plug: 2.35 mm x 0.75 mm\nCenter positive polarity" (at 39.37 55.88 0)
+    (effects (font (size 1.27 1.27)) (justify right bottom))
   )
   (text "*see Note 4" (at 154.94 66.04 0)
     (effects (font (size 1.27 1.27)) (justify right bottom))
   )
-  (text "Main power inputs (DC jack, battery)" (at 134.62 26.67 0)
+  (text "Main power inputs (DC jack, battery)\n0.7W" (at 134.62 29.21 0)
     (effects (font (size 1.27 1.27) (thickness 0.254) bold) (justify right bottom))
   )
@@
   )
   (symbol (lib_id "Device:Battery") (at 105.41 59.69 0) (unit 1)
-    (in_bom yes) (on_board yes) (dnp no)
-    (property "Reference" "BT1" (at 108.1532 58.5216 0)
-      (effects (font (size 1.27 1.27)) (justify left))
-    )
-    (property "Value" "Battery" (at 108.1532 60.833 0)
+    (in_bom yes) (on_board yes) (dnp no) (fields_autoplaced)
+    (property "Reference" "BT1" (at 109.22 57.8485 0)
+      (effects (font (size 1.27 1.27)) (justify left))
+    )
+    (property "Value" "2xAAA" (at 109.22 60.3885 0)
       (effects (font (size 1.27 1.27)) (justify left))
     )
@@
   )
   (symbol (lib_id "Connector:Barrel_Jack_Switch_MountingPin") (at 50.8 54.61 0) (unit 1)
-    (in_bom yes) (on_board yes) (dnp no)
-    (property "Reference" "P4" (at 52.2478 46.5582 0)
-      (effects (font (size 1.27 1.27)))
-    )
-    (property "Value" "DC 3V" (at 52.2478 48.8696 0)
-      (effects (font (size 1.27 1.27)))
-    )
+    (in_bom yes) (on_board yes) (dnp no) (fields_autoplaced)
+    (property "Reference" "P4" (at 50.8 45.72 0)
+      (effects (font (size 1.27 1.27)))
+    )
+    (property "Value" "DC 3V" (at 50.8 48.26 0)
+      (effects (font (size 1.27 1.27)))
+    )

Commit message: Tidy up switch symbols
Parts:
- SW1: symbol Gekkio_Switch:GameBoy_SW_SP3T -> Gekkio_Switch:GameBoy_SW_SP3T_MGB
Changed lines of the file:
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@@
     )
   )
-  (symbol (lib_id "Gekkio_Switch:GameBoy_SW_SP3T") (at 165.1 54.61 0) (mirror y) (unit 1)
-    (in_bom yes) (on_board yes) (dnp no)
-    (property "Reference" "SW1" (at 165.1 47.4218 0)
+  (symbol (lib_id "Gekkio_Switch:GameBoy_SW_SP3T_MGB") (at 165.1 54.61 0) (mirror y) (unit 1)
+    (in_bom yes) (on_board yes) (dnp no) (fields_autoplaced)
+    (property "Reference" "SW1" (at 165.1 46.99 0)
       (effects (font (size 1.27 1.27)))
     )
-    (property "Value" "SP3T" (at 165.1 49.7332 0)
+    (property "Value" "SP3T" (at 165.1 49.53 0)
       (effects (font (size 1.27 1.27)))
     )
