File: MGB-xCPU/joypad.kicad_sch (KiCad schematic)
At the start: 12 parts, among them SW2 LEFT, SW3 UP, SW4 DOWN, SW5 RIGHT, SW6 SELECT, SW7 START, SW8 B, SW9 A

Commit message: Release: MGB-xCPU rev C
Other:
- title: MGB-xCPU - Joypad -> MGB-xCPU
Changed lines of the file:
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@@
   (paper "A4")
   (title_block
-    (title "MGB-xCPU - Joypad")
-    (date "2020-09-19")
-    (rev "B")
+    (title "MGB-xCPU")
+    (date "2022-01-02")
+    (rev "C")
     (company "https://gekkio.fi")
     (comment 1 "https://github.com/gekkio/gb-schematics")
