File: MGB-xCPU/lcd.kicad_sch (KiCad schematic)
At the start: 42 parts, among them P2 LCD FPC, Q1 2SA1576A, U4 IR3E02

Commit message: MGB uses a TN display, not STN
Other:
- note added: "TN LCD bias generation"
- note removed: "STN LCD bias generation"
Changed lines of the file:
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@@
     (effects (font (size 0.762 0.762)) (justify right bottom))
   )
-  (text "STN LCD bias generation" (at 189.23 43.18 180)
+  (text "TN LCD bias generation" (at 189.23 43.18 180)
     (effects (font (size 1.27 1.27) (thickness 0.254) bold) (justify right bottom))
   )

Commit message: Release: MGB-xCPU rev C
Other:
- title: MGB-xCPU - LCD -> MGB-xCPU
Changed lines of the file:
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@@
   (paper "A4")
   (title_block
-    (title "MGB-xCPU - LCD")
-    (date "2020-09-19")
-    (rev "B")
+    (title "MGB-xCPU")
+    (date "2022-01-02")
+    (rev "C")
     (company "https://gekkio.fi")
     (comment 1 "https://github.com/gekkio/gb-schematics")

Commit message: Remove Farad/Henry units
Parts:
- C20, C21, C22, C23, C24: value 1uF -> 1u
- C28: value 10uF -> 10u
- C3: value 47pF -> 47p
Changed lines of the file:
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@@
       (effects (font (size 1.27 1.27)) (justify left))
     )
-    (property "Value" "10uF" (at 49.911 63.373 0)
+    (property "Value" "10u" (at 49.911 63.373 0)
       (effects (font (size 1.27 1.27)) (justify left))
     )
@@
       (effects (font (size 1.27 1.27)) (justify left))
     )
-    (property "Value" "47pF" (at 115.951 60.833 0)
+    (property "Value" "47p" (at 115.951 60.833 0)
       (effects (font (size 1.27 1.27)) (justify left))
     )
@@
       (effects (font (size 1.27 1.27)) (justify left))
     )
-    (property "Value" "1uF" (at 183.261 58.293 0)
+    (property "Value" "1u" (at 183.261 58.293 0)
       (effects (font (size 1.27 1.27)) (justify left))
     )
@@
       (effects (font (size 1.27 1.27)) (justify left))
     )
-    (property "Value" "1uF" (at 162.941 58.293 0)
+    (property "Value" "1u" (at 162.941 58.293 0)
       (effects (font (size 1.27 1.27)) (justify left))
     )
@@
       (effects (font (size 1.27 1.27)) (justify left))
     )
-    (property "Value" "1uF" (at 142.621 58.293 0)
+    (property "Value" "1u" (at 142.621 58.293 0)
       (effects (font (size 1.27 1.27)) (justify left))
     )
@@
       (effects (font (size 1.27 1.27)) (justify left))
     )
-    (property "Value" "1uF" (at 152.781 58.293 0)
+    (property "Value" "1u" (at 152.781 58.293 0)
       (effects (font (size 1.27 1.27)) (justify left))
     )
@@
       (effects (font (size 1.27 1.27)) (justify left))
     )
-    (property "Value" "1uF" (at 173.101 58.293 0)
-      (effects (font (size 1.27 1.27)) (justify left))
-    )
+    (property "Value" "1u" (at 173.101 58.293 0)
+      (effects (font (size 1.27 1.27)) (justify left))
+    )

Commit message: Tidy up potentiometer symbols, add contrast pot symbols
Parts:
- VR2: symbol Device:R_Variable -> Gekkio_Device_Specialized:R_Potentiometer_GameBoy_Contrast_MGB
Connections:
- net GND: now also VR2.MP (MountPin)
- net VR: now also VR2.2
- net at JP1.1 (A), TP64.1: now also VR2.5; no longer VR2.2
Other:
- note removed: "TODO: more specific symbol"
- moved on the sheet: C20, C21, C22, C23, C24, C28, C3, Q1, R1, U4
