File: MGB-xCPU/link_port.kicad_sch (KiCad schematic)
At the start: 9 parts, among them P3 GameBoy_LinkPort

Commit message: Release: MGB-xCPU rev C
Other:
- title: MGB-xCPU - Link port -> MGB-xCPU
Changed lines of the file:
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@@
   (paper "A4")
   (title_block
-    (title "MGB-xCPU - Link port")
-    (date "2020-09-19")
-    (rev "B")
+    (title "MGB-xCPU")
+    (date "2022-01-02")
+    (rev "C")
     (company "https://gekkio.fi")
     (comment 1 "https://github.com/gekkio/gb-schematics")

Commit message: Remove Farad/Henry units
Parts:
- C4, C5, C6, C7: value 100pF -> 100p
- C9: value 10nF -> 10n
Changed lines of the file:
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@@
       (effects (font (size 1.27 1.27)) (justify left))
     )
-    (property "Value" "10nF" (at 216.281 120.523 0)
+    (property "Value" "10n" (at 216.281 120.523 0)
       (effects (font (size 1.27 1.27)) (justify left))
     )
@@
       (effects (font (size 1.27 1.27)) (justify left))
     )
-    (property "Value" "100pF" (at 198.501 120.523 0)
+    (property "Value" "100p" (at 198.501 120.523 0)
       (effects (font (size 1.27 1.27)) (justify left))
     )
@@
       (effects (font (size 1.27 1.27)) (justify left))
     )
-    (property "Value" "100pF" (at 185.801 120.523 0)
+    (property "Value" "100p" (at 185.801 120.523 0)
       (effects (font (size 1.27 1.27)) (justify left))
     )
@@
       (effects (font (size 1.27 1.27)) (justify left))
     )
-    (property "Value" "100pF" (at 173.101 120.523 0)
+    (property "Value" "100p" (at 173.101 120.523 0)
       (effects (font (size 1.27 1.27)) (justify left))
     )
@@
       (effects (font (size 1.27 1.27)) (justify left))
     )
-    (property "Value" "100pF" (at 160.401 120.523 0)
+    (property "Value" "100p" (at 160.401 120.523 0)
       (effects (font (size 1.27 1.27)) (justify left))
     )
