File: AGS-CPU-11/battery.sch (KiCad schematic (older format))
At the start: 32 parts, among them P4 Battery_Cell, Q1 2SB956, U5 MM1581

Commit message: Fix Q1 pinout mistake
Now the circuit actually makes sense! It's basically the reference
circuit from MM1581 datasheet
Parts:
- Q1: symbol Device:Q_PNP_BCE -> Device:Q_PNP_ECB
Other:
- moved on the sheet: Q1, R21, TP115
Changed lines of the file:
@@
 	1    0    0    -1
 $EndComp
-Wire Wire Line
-	3650 1950 3750 1950
-Connection ~ 4750 2150
-Wire Wire Line
-	4750 2150 4250 2150
-Wire Wire Line
-	4750 2050 4750 2150
-Text HLabel 3650 1950 0    50   Input ~ 0
+Text HLabel 3850 1800 0    50   Input ~ 0
 EXT_VIN
 $Comp
 L Device:R R?
 U 1 1 5BE0D3D8
-P 4000 2150
+P 4350 1800
 AR Path="/5BE0D3D8" Ref="R?"  Part="1"
 AR Path="/5BE05CB3/5BE0D3D8" Ref="R21"  Part="1"
-F 0 "R21" V 3793 2150 50  0000 C CNN
-F 1 "680R" V 3884 2150 50  0000 C CNN
-F 2 "" V 3930 2150 50  0001 C CNN
-F 3 "~" H 4000 2150 50  0001 C CNN
-	1    4000 2150
+F 0 "R21" V 4143 1800 50  0000 C CNN
+F 1 "680R" V 4234 1800 50  0000 C CNN
+F 2 "" V 4280 1800 50  0001 C CNN
+F 3 "~" H 4350 1800 50  0001 C CNN
+	1    4350 1800
 	0    -1   1    0
 $EndComp
@@
 L Connector:TestPoint TP?
 U 1 1 5BE0D3CE
-P 4750 2050
+P 4850 2150
 AR Path="/5BE0D3CE" Ref="TP?"  Part="1"
 AR Path="/5BE05CB3/5BE0D3CE" Ref="TP115"  Part="1"
-F 0 "TP115" H 4808 2170 50  0000 L CNN
-F 1 "Q1B" H 4808 2079 50  0000 L CNN
-F 2 "" H 4950 2050 50  0001 C CNN
-F 3 "~" H 4950 2050 50  0001 C CNN
-	1    4750 2050
-	1    0    0    -1
+F 0 "TP115" V 4804 2338 50  0000 L CNN
+F 1 "Q1B" V 4895 2338 50  0000 L CNN
+F 2 "" H 5050 2150 50  0001 C CNN
+F 3 "~" H 5050 2150 50  0001 C CNN
+	1    4850 2150
+	0    1    1    0
 $EndComp
 $Comp
@@
 Connection ~ 4750 2700
 $Comp
-L Device:Q_PNP_BCE Q?
+L Device:Q_PNP_ECB Q?
 U 1 1 5BE0D411
-P 4150 2500
+P 4050 2150
 AR Path="/5BE0D411" Ref="Q?"  Part="1"
 AR Path="/5BE05CB3/5BE0D411" Ref="Q1"  Part="1"
-F 0 "Q1" H 4341 2546 50  0000 L CNN
-F 1 "2SB956" H 4341 2455 50  0000 L CNN
-F 2 "" H 4350 2600 50  0001 C CNN
-F 3 "~" H 4150 2500 50  0001 C CNN
-	1    4150 2500
-	1    0    0    1
+F 0 "Q1" H 4241 2104 50  0000 L CNN
+F 1 "2SB956" H 4241 2195 50  0000 L CNN
+F 2 "" H 4250 2250 50  0001 C CNN
+F 3 "~" H 4050 2150 50  0001 C CNN
+	1    4050 2150
+	-1   0    0    1
 $EndComp
 Wire Wire Line
-	4250 2300 4250 2150
+	3950 1950 3950 1800
 Wire Wire Line
 	4750 2650 4750 2700
-Wire Wire Line
-	4750 2350 4750 2150
-Wire Wire Line
-	3750 1950 3750 2150
-Wire Wire Line
-	3750 2500 3950 2500
-Wire Wire Line
-	4150 2150 4250 2150
-Connection ~ 4250 2150
-Wire Wire Line
-	3850 2150 3750 2150
-Connection ~ 3750 2150
-Wire Wire Line
-	3750 2150 3750 2500
 Wire Wire Line
 	4750 3700 4750 3800
@@
 	5700 3500 5700 3600
 Wire Wire Line
-	4250 2700 4250 3200
+	3950 2350 3950 3200
 Wire Wire Line
 	6200 3200 6200 3100
@@
 	6200 3500 6200 3200
 Wire Wire Line
-	6200 3200 4250 3200
+	6200 3200 3950 3200
 Wire Wire Line
 	3000 3800 3500 3800
@@
 Text HLabel 3600 3500 2    50   Output ~ 0
 VBAT
+Connection ~ 4750 2150
+Wire Wire Line
+	4750 2150 4750 2350
+Wire Wire Line
+	3850 1800 3950 1800
+Wire Wire Line
+	3950 1800 4200 1800
+Connection ~ 3950 1800
+Wire Wire Line
+	4250 2150 4750 2150
+Wire Wire Line
+	4850 2150 4750 2150
+Wire Wire Line
+	4750 1800 4500 1800
+Wire Wire Line
+	4750 1800 4750 2150
 $EndSCHEMATC
