File: AGS-CPU-11/AGS-CPU-11.sch (KiCad schematic (older format))
At the start: 50 parts, among them Q8 DTC114Y, SW1 GameBoy_SW_SPDT, U1 AGB-CPU, U2 AGB-SRAM, X1 4.194304 MHz

Commit message: Fix C2 value
Parts:
- C2: value 34pF -> 33pF
Changed lines of the file:
@@
 P 10300 5950
 F 0 "C2" H 10415 5996 50  0000 L CNN
-F 1 "34pF" H 10415 5905 50  0000 L CNN
+F 1 "33pF" H 10415 5905 50  0000 L CNN
 F 2 "" H 10338 5800 50  0001 C CNN
 F 3 "~" H 10300 5950 50  0001 C CNN
