File: AGS-CPU-11/EXT2.kicad_sch (KiCad schematic)
At the start: 14 parts, among them P3 EXT2, Q11 2SD1819A

Commit message: Hide test point references
Parts:
- TP104, TP105, TP106, TP107, TP108, TP109: symbol Connector:TestPoint -> Connector:TestPoint_Small
Changed lines of the file:
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@@
     (pin "2")
   )
-  (symbol (lib_id "Connector:TestPoint") (at 93.98 62.23 0) (unit 1)
-    (in_bom yes) (on_board yes)
+  (symbol (lib_id "Connector:TestPoint_Small") (at 93.98 62.23 0) (unit 1)
+    (in_bom yes) (on_board yes) (fields_autoplaced)
     (property "Reference" "TP105" (id 0) (at 95.4532 59.182 0)
-      (effects (font (size 1.27 1.27)) (justify left))
-    )
-    (property "Value" "P31" (id 1) (at 95.4532 61.4934 0)
+      (effects (font (size 1.27 1.27)) (justify left) hide)
+    )
+    (property "Value" "P31" (id 1) (at 95.25 62.2299 0)
       (effects (font (size 1.27 1.27)) (justify left))
     )
@@
     (pin "2")
   )
-  (symbol (lib_id "Connector:TestPoint") (at 93.98 73.66 0) (unit 1)
-    (in_bom yes) (on_board yes)
+  (symbol (lib_id "Connector:TestPoint_Small") (at 93.98 73.66 0) (unit 1)
+    (in_bom yes) (on_board yes) (fields_autoplaced)
     (property "Reference" "TP106" (id 0) (at 95.4532 70.612 0)
-      (effects (font (size 1.27 1.27)) (justify left))
-    )
-    (property "Value" "P33" (id 1) (at 95.4532 72.9234 0)
+      (effects (font (size 1.27 1.27)) (justify left) hide)
+    )
+    (property "Value" "P33" (id 1) (at 95.25 73.6599 0)
       (effects (font (size 1.27 1.27)) (justify left))
     )
@@
     (pin "1")
   )
-  (symbol (lib_id "Connector:TestPoint") (at 93.98 85.09 0) (unit 1)
-    (in_bom yes) (on_board yes)
+  (symbol (lib_id "Connector:TestPoint_Small") (at 93.98 85.09 0) (unit 1)
+    (in_bom yes) (on_board yes) (fields_autoplaced)
     (property "Reference" "TP107" (id 0) (at 95.4532 82.042 0)
-      (effects (font (size 1.27 1.27)) (justify left))
-    )
-    (property "Value" "P34" (id 1) (at 95.4532 84.3534 0)
+      (effects (font (size 1.27 1.27)) (justify left) hide)
+    )
+    (property "Value" "P34" (id 1) (at 95.25 85.0899 0)
       (effects (font (size 1.27 1.27)) (justify left))
     )
@@
     (pin "1")
   )
-  (symbol (lib_id "Connector:TestPoint") (at 78.74 100.33 0) (unit 1)
-    (in_bom yes) (on_board yes)
+  (symbol (lib_id "Connector:TestPoint_Small") (at 78.74 100.33 0) (unit 1)
+    (in_bom yes) (on_board yes) (fields_autoplaced)
     (property "Reference" "TP104" (id 0) (at 80.2132 97.282 0)
-      (effects (font (size 1.27 1.27)) (justify left))
-    )
-    (property "Value" "P32" (id 1) (at 80.2132 99.5934 0)
+      (effects (font (size 1.27 1.27)) (justify left) hide)
+    )
+    (property "Value" "P32" (id 1) (at 80.01 100.3299 0)
       (effects (font (size 1.27 1.27)) (justify left))
     )
@@
     (pin "4")
   )
-  (symbol (lib_id "Connector:TestPoint") (at 114.3 130.81 0) (unit 1)
-    (in_bom yes) (on_board yes)
-    (property "Reference" "TP108" (id 0) (at 115.7732 127.762 0)
-      (effects (font (size 1.27 1.27)) (justify left))
-    )
-    (property "Value" "P35" (id 1) (at 115.7732 130.0734 0)
-      (effects (font (size 1.27 1.27)) (justify left))
-    )
-    (property "Footprint" "" (id 2) (at 119.38 130.81 0)
-      (effects (font (size 1.27 1.27)) hide)
-    )
-    (property "Datasheet" "~" (id 3) (at 119.38 130.81 0)
+  (symbol (lib_id "Connector:TestPoint_Small") (at 114.3 130.81 90) (unit 1)
+    (in_bom yes) (on_board yes) (fields_autoplaced)
+    (property "Reference" "TP108" (id 0) (at 111.252 129.3368 0)
+      (effects (font (size 1.27 1.27)) (justify left) hide)
+    )
+    (property "Value" "P35" (id 1) (at 114.3 128.27 90))
+    (property "Footprint" "" (id 2) (at 114.3 125.73 0)
+      (effects (font (size 1.27 1.27)) hide)
+    )
+    (property "Datasheet" "~" (id 3) (at 114.3 125.73 0)
       (effects (font (size 1.27 1.27)) hide)
     )
@@
     (pin "1")
   )
-  (symbol (lib_id "Connector:TestPoint") (at 134.62 121.92 0) (unit 1)
-    (in_bom yes) (on_board yes)
-    (property "Reference" "TP109" (id 0) (at 136.0932 118.9228 0)
-      (effects (font (size 1.27 1.27)) (justify left))
-    )
-    (property "Value" "SW" (id 1) (at 136.0932 121.2342 0)
-      (effects (font (size 1.27 1.27)) (justify left))
-    )
-    (property "Footprint" "" (id 2) (at 139.7 121.92 0)
-      (effects (font (size 1.27 1.27)) hide)
-    )
-    (property "Datasheet" "~" (id 3) (at 139.7 121.92 0)
-      (effects (font (size 1.27 1.27)) hide)
-    )
+  (symbol (lib_id "Connector:TestPoint_Small") (at 134.62 121.92 90) (unit 1)
+    (in_bom yes) (on_board yes) (fields_autoplaced)
+    (property "Reference" "TP109" (id 0) (at 131.6228 120.4468 0)
+      (effects (font (size 1.27 1.27)) (justify left) hide)
+    )
+    (property "Value" "SW" (id 1) (at 134.62 119.38 90))
+    (property "Footprint" "" (id 2) (at 134.62 116.84 0)
+      (effects (font (size 1.27 1.27)) hide)
+    )
+    (property "Datasheet" "~" (id 3) (at 134.62 116.84 0)
+      (effects (font (size 1.27 1.27)) hide)
+    )

Commit message: Release: AGB-CPU-11 rev D
Other:
- title: AGS-CPU-11 - EXT2 port -> AGS-CPU-11
Changed lines of the file:
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@@
   (paper "A4")
   (title_block
-    (title "AGS-CPU-11 - EXT2 port")
-    (date "2021-07-26")
-    (rev "C")
+    (title "AGS-CPU-11")
+    (date "2022-01-02")
+    (rev "D")
     (company "https://gekkio.fi")
     (comment 1 "https://github.com/Gekkio/gb-schematics")
