File: AGS-CPU-11/leds.kicad_sch (KiCad schematic)
At the start: 14 parts, among them Q2 DTA144W, Q4 DTA144W, Q6 2SD1819A

Commit message: Hide test point references
Parts:
- TP100, TP101, TP102, TP103: symbol Connector:TestPoint -> Connector:TestPoint_Small
Changed lines of the file:
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@@
   (junction (at 41.91 86.36) (diameter 0) (color 0 0 0 0)
   )
+  (junction (at 114.3 101.6) (diameter 0) (color 0 0 0 0)
+  )
+  (junction (at 106.68 76.2) (diameter 0) (color 0 0 0 0)
+  )
   (junction (at 63.5 101.6) (diameter 0) (color 0 0 0 0)
   )
-  (junction (at 106.68 76.2) (diameter 0) (color 0 0 0 0)
-  )
-  (junction (at 114.3 101.6) (diameter 0) (color 0 0 0 0)
-  )
   (polyline (pts (xy 44.45 116.84) (xy 82.55 116.84))
     (stroke (width 0.3) (type default) (color 0 0 0 0))
@@
     (stroke (width 0) (type default) (color 0 0 0 0))
   )
+  (wire (pts (xy 175.26 101.6) (xy 177.8 101.6))
+    (stroke (width 0) (type default) (color 0 0 0 0))
+  )
   (wire (pts (xy 114.3 86.36) (xy 114.3 87.63))
     (stroke (width 0) (type default) (color 0 0 0 0))
@@
   (polyline (pts (xy 158.75 116.84) (xy 158.75 63.5))
     (stroke (width 0.3) (type default) (color 0 0 0 0))
+  )
+  (wire (pts (xy 60.96 101.6) (xy 63.5 101.6))
+    (stroke (width 0) (type default) (color 0 0 0 0))
+  )
+  (wire (pts (xy 111.76 101.6) (xy 114.3 101.6))
+    (stroke (width 0) (type default) (color 0 0 0 0))
   )
   (wire (pts (xy 114.3 87.63) (xy 114.3 88.9))
@@
     (pin "1")
   )
-  (symbol (lib_id "Connector:TestPoint") (at 63.5 101.6 90) (unit 1)
-    (in_bom yes) (on_board yes)
-    (property "Reference" "TP100" (id 0) (at 58.7502 100.4316 90)
-      (effects (font (size 1.27 1.27)) (justify left))
-    )
-    (property "Value" "DL1A" (id 1) (at 58.7502 102.743 90)
-      (effects (font (size 1.27 1.27)) (justify left))
-    )
-    (property "Footprint" "" (id 2) (at 63.5 96.52 0)
-      (effects (font (size 1.27 1.27)) hide)
-    )
-    (property "Datasheet" "~" (id 3) (at 63.5 96.52 0)
+  (symbol (lib_id "Connector:TestPoint_Small") (at 60.96 101.6 90) (unit 1)
+    (in_bom yes) (on_board yes) (fields_autoplaced)
+    (property "Reference" "TP100" (id 0) (at 56.2102 100.4316 90)
+      (effects (font (size 1.27 1.27)) (justify left) hide)
+    )
+    (property "Value" "DL1A" (id 1) (at 59.69 101.5999 90)
+      (effects (font (size 1.27 1.27)) (justify left))
+    )
+    (property "Footprint" "" (id 2) (at 60.96 96.52 0)
+      (effects (font (size 1.27 1.27)) hide)
+    )
+    (property "Datasheet" "~" (id 3) (at 60.96 96.52 0)
       (effects (font (size 1.27 1.27)) hide)
     )
@@
     (pin "1")
   )
-  (symbol (lib_id "Connector:TestPoint") (at 123.19 87.63 0) (unit 1)
-    (in_bom yes) (on_board yes)
+  (symbol (lib_id "Connector:TestPoint_Small") (at 123.19 87.63 0) (unit 1)
+    (in_bom yes) (on_board yes) (fields_autoplaced)
     (property "Reference" "TP102" (id 0) (at 124.6632 84.6328 0)
-      (effects (font (size 1.27 1.27)) (justify left))
-    )
-    (property "Value" "Q6C" (id 1) (at 124.6632 86.9442 0)
+      (effects (font (size 1.27 1.27)) (justify left) hide)
+    )
+    (property "Value" "Q6C" (id 1) (at 124.46 87.6299 0)
       (effects (font (size 1.27 1.27)) (justify left))
     )
@@
     (pin "2")
   )
-  (symbol (lib_id "Connector:TestPoint") (at 114.3 101.6 90) (unit 1)
-    (in_bom yes) (on_board yes)
-    (property "Reference" "TP101" (id 0) (at 109.5502 100.4316 90)
-      (effects (font (size 1.27 1.27)) (justify left))
-    )
-    (property "Value" "DL2A" (id 1) (at 109.5502 102.743 90)
-      (effects (font (size 1.27 1.27)) (justify left))
-    )
-    (property "Footprint" "" (id 2) (at 114.3 96.52 0)
-      (effects (font (size 1.27 1.27)) hide)
-    )
-    (property "Datasheet" "~" (id 3) (at 114.3 96.52 0)
+  (symbol (lib_id "Connector:TestPoint_Small") (at 111.76 101.6 90) (unit 1)
+    (in_bom yes) (on_board yes) (fields_autoplaced)
+    (property "Reference" "TP101" (id 0) (at 111.76 96.52 90)
+      (effects (font (size 1.27 1.27)) hide)
+    )
+    (property "Value" "DL2A" (id 1) (at 110.49 101.5999 90)
+      (effects (font (size 1.27 1.27)) (justify left))
+    )
+    (property "Footprint" "" (id 2) (at 111.76 96.52 0)
+      (effects (font (size 1.27 1.27)) hide)
+    )
+    (property "Datasheet" "~" (id 3) (at 111.76 96.52 0)
       (effects (font (size 1.27 1.27)) hide)
     )
@@
     (pin "1")
   )
-  (symbol (lib_id "Connector:TestPoint") (at 177.8 101.6 90) (unit 1)
-    (in_bom yes) (on_board yes)
-    (property "Reference" "TP103" (id 0) (at 173.0502 100.4316 90)
-      (effects (font (size 1.27 1.27)) (justify left))
-    )
-    (property "Value" "DL3A" (id 1) (at 173.0502 102.743 90)
-      (effects (font (size 1.27 1.27)) (justify left))
-    )
-    (property "Footprint" "" (id 2) (at 177.8 96.52 0)
-      (effects (font (size 1.27 1.27)) hide)
-    )
-    (property "Datasheet" "~" (id 3) (at 177.8 96.52 0)
-      (effects (font (size 1.27 1.27)) hide)
-    )
+  (symbol (lib_id "Connector:TestPoint_Small") (at 175.26 101.6 90) (unit 1)
+    (in_bom yes) (on_board yes) (fields_autoplaced)
+    (property "Reference" "TP103" (id 0) (at 170.5102 100.4316 90)
+      (effects (font (size 1.27 1.27)) (justify left) hide)
+    )
+    (property "Value" "DL3A" (id 1) (at 173.99 101.5999 90)
+      (effects (font (size 1.27 1.27)) (justify left))
+    )
+    (property "Footprint" "" (id 2) (at 175.26 96.52 0)
+      (effects (font (size 1.27 1.27)) hide)
+    )
+    (property "Datasheet" "~" (id 3) (at 175.26 96.52 0)
+      (effects (font (size 1.27 1.27)) hide)
+    )

Commit message: Release: AGB-CPU-11 rev D
Other:
- title: AGS-CPU-11 - LEDs -> AGS-CPU-11
Changed lines of the file:
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@@
   (paper "A4")
   (title_block
-    (title "AGS-CPU-11 - LEDs")
-    (date "2021-07-26")
-    (rev "C")
+    (title "AGS-CPU-11")
+    (date "2022-01-02")
+    (rev "D")
     (company "https://gekkio.fi")
     (comment 1 "https://github.com/Gekkio/gb-schematics")
