File: AGS-CPU-11/EXT1.kicad_sch (KiCad schematic)
At the start: 9 parts, among them P5 EXT1

Commit message: Release: AGB-CPU-11 rev D
Other:
- title: AGS-CPU-11 - EXT1 port -> AGS-CPU-11
Changed lines of the file:
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@@
   (paper "A4")
   (title_block
-    (title "AGS-CPU-11 - EXT1 port")
-    (date "2021-07-26")
-    (rev "C")
+    (title "AGS-CPU-11")
+    (date "2022-01-02")
+    (rev "D")
     (company "https://gekkio.fi")
     (comment 1 "https://github.com/Gekkio/gb-schematics")

Commit message: Remove Farad/Henry units
Parts:
- C10, C8, C9: value 100pF -> 100p
- C7: value 2.2uF -> 2.2u
Changed lines of the file:
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@@
       (effects (font (size 1.27 1.27)) (justify right))
     )
-    (property "Value" "2.2uF" (at 179.9844 109.093 0)
+    (property "Value" "2.2u" (at 179.9844 109.093 0)
       (effects (font (size 1.27 1.27)) (justify right))
     )
@@
       (effects (font (size 1.27 1.27)) (justify left))
     )
-    (property "Value" "100pF" (at 101.981 109.093 0)
+    (property "Value" "100p" (at 101.981 109.093 0)
       (effects (font (size 1.27 1.27)) (justify left))
     )
@@
       (effects (font (size 1.27 1.27)) (justify left))
     )
-    (property "Value" "100pF" (at 113.411 109.093 0)
+    (property "Value" "100p" (at 113.411 109.093 0)
       (effects (font (size 1.27 1.27)) (justify left))
     )
@@
       (effects (font (size 1.27 1.27)) (justify left))
     )
-    (property "Value" "100pF" (at 124.841 109.093 0)
+    (property "Value" "100p" (at 124.841 109.093 0)
       (effects (font (size 1.27 1.27)) (justify left))
     )
