File: AGS-CPU-11/audio_amp.kicad_sch (KiCad schematic)
At the start: 43 parts, among them U3 AGB-AMP, U9 RN4986

Commit message: Hide test point references
Parts:
- TP51, TP52, TP53, TP54, TP55, TP56, TP57, TP58, TP59, TP60, TP61, TP62, TP63, TP64, TP65, TP66: symbol Connector:TestPoint -> Connector:TestPoint_Small

Commit message: Release: AGB-CPU-11 rev D
Other:
- title: AGS-CPU-11 - Audio amplifier -> AGS-CPU-11
Changed lines of the file:
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@@
   (paper "A4")
   (title_block
-    (title "AGS-CPU-11 - Audio amplifier")
-    (date "2021-07-26")
-    (rev "C")
+    (title "AGS-CPU-11")
+    (date "2022-01-02")
+    (rev "D")
     (company "https://gekkio.fi")
     (comment 1 "https://github.com/Gekkio/gb-schematics")

Commit message: Remove Farad/Henry units
Parts:
- C14, C17: value 560pF -> 560p
- C15, C18: value 100pF -> 100p
- C16, C19: value 1nF -> 1n
- C20, C21, C22, C23, C25, C26, C27: value 100nF -> 100n
- C24: value 1uF -> 1u
Changed lines of the file:
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@@
       (effects (font (size 1.27 1.27)) (justify left))
     )
-    (property "Value" "1uF" (at 178.181 124.333 0)
+    (property "Value" "1u" (at 178.181 124.333 0)
       (effects (font (size 1.27 1.27)) (justify left))
     )
@@
       (effects (font (size 1.27 1.27)) (justify left))
     )
-    (property "Value" "100pF" (at 63.881 129.413 0)
+    (property "Value" "100p" (at 63.881 129.413 0)
       (effects (font (size 1.27 1.27)) (justify left))
     )
@@
       (effects (font (size 1.27 1.27)) (justify left))
     )
-    (property "Value" "100pF" (at 38.481 129.413 0)
+    (property "Value" "100p" (at 38.481 129.413 0)
       (effects (font (size 1.27 1.27)) (justify left))
     )
@@
       (effects (font (size 1.27 1.27)) (justify left))
     )
-    (property "Value" "1nF" (at 51.181 129.413 0)
+    (property "Value" "1n" (at 51.181 129.413 0)
       (effects (font (size 1.27 1.27)) (justify left))
     )
@@
       (effects (font (size 1.27 1.27)) (justify left))
     )
-    (property "Value" "560pF" (at 51.181 110.363 0)
+    (property "Value" "560p" (at 51.181 110.363 0)
       (effects (font (size 1.27 1.27)) (justify left))
     )
@@
       (effects (font (size 1.27 1.27)) (justify left))
     )
-    (property "Value" "560pF" (at 76.581 110.363 0)
+    (property "Value" "560p" (at 76.581 110.363 0)
       (effects (font (size 1.27 1.27)) (justify left))
     )
@@
       (effects (font (size 1.27 1.27)) (justify left))
     )
-    (property "Value" "100nF" (at 189.611 124.333 0)
+    (property "Value" "100n" (at 189.611 124.333 0)
       (effects (font (size 1.27 1.27)) (justify left))
     )
@@
       (effects (font (size 1.27 1.27)) (justify left))
     )
-    (property "Value" "100nF" (at 137.541 129.413 0)
+    (property "Value" "100n" (at 137.541 129.413 0)
       (effects (font (size 1.27 1.27)) (justify left))
     )
@@
       (effects (font (size 1.27 1.27)) (justify left))
     )
-    (property "Value" "1nF" (at 76.581 129.413 0)
+    (property "Value" "1n" (at 76.581 129.413 0)
       (effects (font (size 1.27 1.27)) (justify left))
     )
@@
       (effects (font (size 1.27 1.27)) (justify left))
     )
-    (property "Value" "100nF" (at 202.311 124.333 0)
+    (property "Value" "100n" (at 202.311 124.333 0)
       (effects (font (size 1.27 1.27)) (justify left))
     )
@@
       (effects (font (size 1.27 1.27)) (justify left))
     )
-    (property "Value" "100nF" (at 215.011 124.333 0)
+    (property "Value" "100n" (at 215.011 124.333 0)
       (effects (font (size 1.27 1.27)) (justify left))
     )
@@
       (effects (font (size 1.27 1.27)) (justify left))
     )
-    (property "Value" "100nF" (at 227.711 124.333 0)
+    (property "Value" "100n" (at 227.711 124.333 0)
       (effects (font (size 1.27 1.27)) (justify left))
     )
@@
       (effects (font (size 1.27 1.27)) (justify left))
     )
-    (property "Value" "100nF" (at 165.481 152.273 0)
+    (property "Value" "100n" (at 165.481 152.273 0)
       (effects (font (size 1.27 1.27)) (justify left))
     )
@@
       (effects (font (size 1.27 1.27)) (justify left))
     )
-    (property "Value" "100nF" (at 152.781 152.273 0)
-      (effects (font (size 1.27 1.27)) (justify left))
-    )
+    (property "Value" "100n" (at 152.781 152.273 0)
+      (effects (font (size 1.27 1.27)) (justify left))
+    )
