File: AGS-CPU-11/battery.kicad_sch (KiCad schematic)
At the start: 32 parts, among them P4 Battery_Cell, Q1 2SB956, U5 MM1581

Commit message: Hide test point references
Parts:
- TP110, TP111, TP112, TP113, TP114, TP115, TP116, TP117, TP118, TP119, TP120, TP121: symbol Connector:TestPoint -> Connector:TestPoint_Small

Commit message: Release: AGB-CPU-11 rev D
Other:
- title: AGS-CPU-11 - Battery -> AGS-CPU-11
Changed lines of the file:
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@@
   (paper "A4")
   (title_block
-    (title "AGS-CPU-11 - Battery")
-    (date "2021-07-26")
-    (rev "C")
+    (title "AGS-CPU-11")
+    (date "2022-01-02")
+    (rev "D")
     (company "https://gekkio.fi")
     (comment 1 "https://github.com/Gekkio/gb-schematics")

Commit message: Remove Farad/Henry units
Parts:
- C28: value 1uF -> 1u
- C31, C68, C71, C75: value 100nF -> 100n
Changed lines of the file:
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@@
       (effects (font (size 1.27 1.27)) (justify left))
     )
-    (property "Value" "100nF" (at 123.571 76.073 0)
+    (property "Value" "100n" (at 123.571 76.073 0)
       (effects (font (size 1.27 1.27)) (justify left))
     )
@@
       (effects (font (size 1.27 1.27)) (justify left))
     )
-    (property "Value" "1uF" (at 112.141 124.333 0)
+    (property "Value" "1u" (at 112.141 124.333 0)
       (effects (font (size 1.27 1.27)) (justify left))
     )
@@
       (effects (font (size 1.27 1.27)) (justify left))
     )
-    (property "Value" "100nF" (at 162.941 124.333 0)
+    (property "Value" "100n" (at 162.941 124.333 0)
       (effects (font (size 1.27 1.27)) (justify left))
     )
@@
       (effects (font (size 1.27 1.27)) (justify left))
     )
-    (property "Value" "100nF" (at 218.821 123.063 0)
+    (property "Value" "100n" (at 218.821 123.063 0)
       (effects (font (size 1.27 1.27)) (justify left))
     )
@@
       (effects (font (size 1.27 1.27)) (justify left))
     )
-    (property "Value" "100nF" (at 79.121 101.473 0)
-      (effects (font (size 1.27 1.27)) (justify left))
-    )
+    (property "Value" "100n" (at 79.121 101.473 0)
+      (effects (font (size 1.27 1.27)) (justify left))
+    )
