File: AGS-CPU-11/joypad.kicad_sch (KiCad schematic)
At the start: 24 parts, among them SW10 UP, SW11 DOWN, SW12 RIGHT, SW3 L, SW4 R, SW5 A, SW6 B, SW7 START, SW8 SELECT, SW9 LEFT

Commit message: Hide test point references
Parts:
- TP36, TP37, TP38, TP39, TP40, TP41, TP42, TP43, TP44, TP45: symbol Connector:TestPoint -> Connector:TestPoint_Small

Commit message: Release: AGB-CPU-11 rev D
Other:
- title: AGS-CPU-11 - Joypad -> AGS-CPU-11
Changed lines of the file:
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@@
   (paper "A4")
   (title_block
-    (title "AGS-CPU-11 - Joypad")
-    (date "2021-07-26")
-    (rev "C")
+    (title "AGS-CPU-11")
+    (date "2022-01-02")
+    (rev "D")
     (company "https://gekkio.fi")
     (comment 1 "https://github.com/Gekkio/gb-schematics")

Commit message: Remove Farad/Henry units
Parts:
- C73, C74: value 10nF -> 10n
Changed lines of the file:
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@@
       (effects (font (size 1.27 1.27)) (justify left))
     )
-    (property "Value" "10nF" (at 49.911 49.403 0)
+    (property "Value" "10n" (at 49.911 49.403 0)
       (effects (font (size 1.27 1.27)) (justify left))
     )
@@
       (effects (font (size 1.27 1.27)) (justify left))
     )
-    (property "Value" "10nF" (at 176.911 49.403 0)
+    (property "Value" "10n" (at 176.911 49.403 0)
       (effects (font (size 1.27 1.27)) (justify left))
     )
