File: AGS-CPU-11/lcd.kicad_sch (KiCad schematic)
At the start: 56 parts, among them P2 LCD, Q12 DTA114T, Q7 DTA114T, SW2 LIGHT ON, U6 NL17SZ74, U8 XP04501

Commit message: Hide test point references
Parts:
- TP67, TP68, TP69, TP70, TP71, TP72, TP73, TP74, TP75, TP76, TP77, TP78, TP79, TP80, TP81, TP82, TP83, TP84, TP85, TP86, TP87, TP88, TP89, TP90, TP91, TP92, TP93, TP94, TP95, TP96, TP97, TP98, TP99: symbol Connector:TestPoint -> Connector:TestPoint_Small
Other:
- moved on the sheet: SW2

Commit message: Release: AGB-CPU-11 rev D
Other:
- title: AGS-CPU-11 - LCD -> AGS-CPU-11
Changed lines of the file:
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@@
   (paper "A4")
   (title_block
-    (title "AGS-CPU-11 - LCD")
-    (date "2021-07-26")
-    (rev "C")
+    (title "AGS-CPU-11")
+    (date "2022-01-02")
+    (rev "D")
     (company "https://gekkio.fi")
     (comment 1 "https://github.com/Gekkio/gb-schematics")

Commit message: Remove Farad/Henry units
Parts:
- C11, C12, C70, C77: value 100nF -> 100n
- C69: value 1uF -> 1u
Changed lines of the file:
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@@
       (effects (font (size 1.27 1.27)) (justify left))
     )
-    (property "Value" "100nF" (at 235.331 39.243 0)
+    (property "Value" "100n" (at 235.331 39.243 0)
       (effects (font (size 1.27 1.27)) (justify left))
     )
@@
       (effects (font (size 1.27 1.27)) (justify left))
     )
-    (property "Value" "100nF" (at 201.041 140.843 0)
+    (property "Value" "100n" (at 201.041 140.843 0)
       (effects (font (size 1.27 1.27)) (justify left))
     )
@@
       (effects (font (size 1.27 1.27)) (justify left))
     )
-    (property "Value" "1uF" (at 75.311 55.753 0)
+    (property "Value" "1u" (at 75.311 55.753 0)
       (effects (font (size 1.27 1.27)) (justify left))
     )
@@
       (effects (font (size 1.27 1.27)) (justify left))
     )
-    (property "Value" "100nF" (at 30.861 176.403 0)
+    (property "Value" "100n" (at 30.861 176.403 0)
       (effects (font (size 1.27 1.27)) (justify left))
     )
@@
       (effects (font (size 1.27 1.27)) (justify left))
     )
-    (property "Value" "100nF" (at 65.151 185.293 0)
-      (effects (font (size 1.27 1.27)) (justify left))
-    )
+    (property "Value" "100n" (at 65.151 185.293 0)
+      (effects (font (size 1.27 1.27)) (justify left))
+    )
