File: AGS-CPU-11/power.kicad_sch (KiCad schematic)
At the start: 64 parts, among them Q3 2SK3663, Q5 2SJ647, T1 GameBoy_Transformer_AGS, U4 Conn_02x08_Counter_Clockwise, U7 ???

Commit message: Hide test point references
Parts:
- TP12, TP13, TP14, TP15, TP16, TP17, TP18, TP19, TP20, TP21, TP22, TP23, TP24, TP25, TP26, TP27, TP28, TP29, TP30, TP31, TP32, TP33, TP34, TP35: symbol Connector:TestPoint -> Connector:TestPoint_Small
Connections:
- net VCC: now also U7.4 (S); no longer U7.1 (S)
- net VDRV3: now also U7.5 (G); no longer U7.2 (G)
- net at D3.1 (K), L1.2, TP30.1: now also U7.3 (D); no longer U7.6 (D)

Commit message: Add chip label
Parts:
- U4: value Conn_02x08_Counter_Clockwise -> S6403/9753
Changed lines of the file:
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@@
     (in_bom yes) (on_board yes)
     (property "Reference" "U4" (id 0) (at 73.66 35.1282 0))
-    (property "Value" "Conn_02x08_Counter_Clockwise" (id 1) (at 73.66 37.4396 0))
+    (property "Value" "S6403/9753" (id 1) (at 73.66 37.4396 0))
     (property "Footprint" "" (id 2) (at 72.39 48.26 0)
       (effects (font (size 1.27 1.27)) hide)

Commit message: Release: AGB-CPU-11 rev D
Other:
- title: AGS-CPU-11 - Power -> AGS-CPU-11
Changed lines of the file:
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@@
   (paper "A4")
   (title_block
-    (title "AGS-CPU-11 - Power")
-    (date "2021-07-26")
-    (rev "C")
+    (title "AGS-CPU-11")
+    (date "2022-01-02")
+    (rev "D")
     (company "https://gekkio.fi")
     (comment 1 "https://github.com/Gekkio/gb-schematics")

Commit message: Remove Farad/Henry units
Parts:
- C13: value 100nF -> 100n
- C32, C36, C45, C46, C72: value 1uF -> 1u
- C33: value 47nF -> 47n
- C34: value 470pF -> 470p
- C37, C38, C39: value 4.7uF -> 4.7u
- C40, C42: value 10uF -> 10u
- C41: value 22uF -> 22u
- C43, C44: value 470nF -> 470n
- L1: value 33uH -> 33u
- L2: value 100uH -> 100u
Changed lines of the file:
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@@
       (effects (font (size 1.27 1.27)) (justify left))
     )
-    (property "Value" "10uF" (at 70.7644 182.753 0)
+    (property "Value" "10u" (at 70.7644 182.753 0)
       (effects (font (size 1.27 1.27)) (justify left))
     )
@@
       (effects (font (size 1.27 1.27)))
     )
-    (property "Value" "1uF" (at 116.84 41.6306 90)
+    (property "Value" "1u" (at 116.84 41.6306 90)
       (effects (font (size 1.27 1.27)))
     )
@@
       (effects (font (size 1.27 1.27)) (justify left))
     )
-    (property "Value" "1uF" (at 110.871 68.453 0)
+    (property "Value" "1u" (at 110.871 68.453 0)
       (effects (font (size 1.27 1.27)) (justify left))
     )
@@
       (effects (font (size 1.27 1.27)) (justify right))
     )
-    (property "Value" "4.7uF" (at 138.811 74.803 0)
+    (property "Value" "4.7u" (at 138.811 74.803 0)
       (effects (font (size 1.27 1.27)) (justify right))
     )
@@
       (effects (font (size 1.27 1.27)) (justify left))
     )
-    (property "Value" "10uF" (at 249.809 152.273 0)
+    (property "Value" "10u" (at 249.809 152.273 0)
       (effects (font (size 1.27 1.27)) (justify left))
     )
@@
       (effects (font (size 1.27 1.27)))
     )
-    (property "Value" "100uH" (at 246.38 137.1854 90)
+    (property "Value" "100u" (at 246.38 137.1854 90)
       (effects (font (size 1.27 1.27)))
     )
@@
       (effects (font (size 1.27 1.27)) (justify left))
     )
-    (property "Value" "1uF" (at 67.691 68.453 0)
+    (property "Value" "1u" (at 67.691 68.453 0)
       (effects (font (size 1.27 1.27)) (justify left))
     )
@@
       (effects (font (size 1.27 1.27)) (justify left))
     )
-    (property "Value" "22uF" (at 249.809 101.473 0)
+    (property "Value" "22u" (at 249.809 101.473 0)
       (effects (font (size 1.27 1.27)) (justify left))
     )
@@
       (effects (font (size 1.27 1.27)))
     )
-    (property "Value" "33uH" (at 246.38 86.3854 90)
+    (property "Value" "33u" (at 246.38 86.3854 90)
       (effects (font (size 1.27 1.27)))
     )
@@
       (effects (font (size 1.27 1.27)) (justify left))
     )
-    (property "Value" "1uF" (at 159.131 145.923 0)
+    (property "Value" "1u" (at 159.131 145.923 0)
       (effects (font (size 1.27 1.27)) (justify left))
     )
@@
       (effects (font (size 1.27 1.27)) (justify left))
     )
-    (property "Value" "100nF" (at 169.291 115.443 0)
+    (property "Value" "100n" (at 169.291 115.443 0)
       (effects (font (size 1.27 1.27)) (justify left))
     )
@@
       (effects (font (size 1.27 1.27)) (justify left))
     )
-    (property "Value" "1uF" (at 159.131 115.443 0)
+    (property "Value" "1u" (at 159.131 115.443 0)
       (effects (font (size 1.27 1.27)) (justify left))
     )
@@
       (effects (font (size 1.27 1.27)))
     )
-    (property "Value" "470nF" (at 121.92 147.3454 90)
+    (property "Value" "470n" (at 121.92 147.3454 90)
       (effects (font (size 1.27 1.27)))
     )
@@
       (effects (font (size 1.27 1.27)))
     )
-    (property "Value" "470nF" (at 121.92 116.8654 90)
+    (property "Value" "470n" (at 121.92 116.8654 90)
       (effects (font (size 1.27 1.27)))
     )
@@
       (effects (font (size 1.27 1.27)) (justify right))
     )
-    (property "Value" "4.7uF" (at 58.0644 133.223 0)
+    (property "Value" "4.7u" (at 58.0644 133.223 0)
       (effects (font (size 1.27 1.27)) (justify right))
     )
@@
       (effects (font (size 1.27 1.27)) (justify left))
     )
-    (property "Value" "470pF" (at 54.991 68.453 0)
+    (property "Value" "470p" (at 54.991 68.453 0)
       (effects (font (size 1.27 1.27)) (justify left))
     )
@@
       (effects (font (size 1.27 1.27)) (justify left))
     )
-    (property "Value" "47nF" (at 42.291 68.453 0)
+    (property "Value" "47n" (at 42.291 68.453 0)
       (effects (font (size 1.27 1.27)) (justify left))
     )
@@
       (effects (font (size 1.27 1.27)) (justify right))
     )
-    (property "Value" "4.7uF" (at 126.0856 74.803 0)
+    (property "Value" "4.7u" (at 126.0856 74.803 0)
       (effects (font (size 1.27 1.27)) (justify right))
     )
