File: AGS-CPU-11/AGS-CPU-11.kicad_sch (KiCad schematic)
At the start: 50 parts, among them Q8 DTC114Y, SW1 GameBoy_SW_SPDT, U1 CPU AGB B, U2 AGB-SRAM, X1 4.194304 MHz

Commit message: Hide test point references
Parts:
- TP1, TP10, TP11, TP2, TP3, TP4, TP5, TP6, TP7, TP8, TP9: symbol Connector:TestPoint -> Connector:TestPoint_Small

Commit message: Add electrolytic capacitor rating
Parts:
- CP1: Rating (none) -> 4V
Changed lines of the file:
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@@
   )
   (symbol (lib_id "Device:C_Polarized") (at 44.45 101.6 0) (mirror y) (unit 1)
-    (in_bom yes) (on_board yes)
-    (property "Reference" "CP1" (id 0) (at 41.4528 100.4316 0)
-      (effects (font (size 1.27 1.27)) (justify left))
+    (in_bom yes) (on_board yes) (fields_autoplaced)
+    (property "Reference" "CP1" (id 0) (at 48.26 98.1709 0)
+      (effects (font (size 1.27 1.27)) (justify right))
     )
-    (property "Value" "100uF" (id 1) (at 41.4528 102.743 0)
-      (effects (font (size 1.27 1.27)) (justify left))
+    (property "Value" "100uF" (id 1) (at 48.26 100.7109 0)
+      (effects (font (size 1.27 1.27)) (justify right))
     )
     (property "Footprint" "" (id 2) (at 43.4848 105.41 0)
@@
       (effects (font (size 1.27 1.27)) hide)
     )
+    (property "Rating" "4V" (id 4) (at 48.26 103.2509 0)
+      (effects (font (size 1.27 1.27)) (justify right))
+    )
     (pin "1")

Commit message: Remove Farad/Henry units
Parts:
- C1: value 27pF -> 27p
- C2: value 33pF -> 33p
- C4: value 680nF -> 680n
- C47, C48, C49, C50: value 10nF -> 10n
- C5: value 1uF -> 1u
- C51, C52, C53, C54, C55, C56, C57, C58, C59, C6, C60, C61, C62, C63, C64, C65, C66, C67: value 100nF -> 100n
- CP1: value 100uF -> 100u
Changed lines of the file:
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@@
       (effects (font (size 1.27 1.27)) (justify right))
     )
-    (property "Value" "100uF" (at 48.26 100.7109 0)
+    (property "Value" "100u" (at 48.26 100.7109 0)
       (effects (font (size 1.27 1.27)) (justify right))
     )
@@
       (effects (font (size 1.27 1.27)) (justify left))
     )
-    (property "Value" "100nF" (at 235.331 98.933 0)
+    (property "Value" "100n" (at 235.331 98.933 0)
       (effects (font (size 1.27 1.27)) (justify left))
     )
@@
       (effects (font (size 1.27 1.27)) (justify right))
     )
-    (property "Value" "27pF" (at 240.9444 152.273 0)
+    (property "Value" "27p" (at 240.9444 152.273 0)
       (effects (font (size 1.27 1.27)) (justify right))
     )
@@
       (effects (font (size 1.27 1.27)) (justify left))
     )
-    (property "Value" "33pF" (at 264.541 152.273 0)
+    (property "Value" "33p" (at 264.541 152.273 0)
       (effects (font (size 1.27 1.27)) (justify left))
     )
@@
       (effects (font (size 1.27 1.27)) (justify left))
     )
-    (property "Value" "1uF" (at 28.321 137.033 0)
+    (property "Value" "1u" (at 28.321 137.033 0)
       (effects (font (size 1.27 1.27)) (justify left))
     )
@@
       (effects (font (size 1.27 1.27)) (justify left))
     )
-    (property "Value" "680nF" (at 56.261 143.383 0)
+    (property "Value" "680n" (at 56.261 143.383 0)
       (effects (font (size 1.27 1.27)) (justify left))
     )
@@
       (effects (font (size 1.27 1.27)) (justify left))
     )
-    (property "Value" "10nF" (at 23.241 167.513 0)
+    (property "Value" "10n" (at 23.241 167.513 0)
       (effects (font (size 1.27 1.27)) (justify left))
     )
@@
       (effects (font (size 1.27 1.27)) (justify left))
     )
-    (property "Value" "10nF" (at 35.941 167.513 0)
+    (property "Value" "10n" (at 35.941 167.513 0)
       (effects (font (size 1.27 1.27)) (justify left))
     )
@@
       (effects (font (size 1.27 1.27)) (justify left))
     )
-    (property "Value" "10nF" (at 61.341 167.513 0)
+    (property "Value" "10n" (at 61.341 167.513 0)
       (effects (font (size 1.27 1.27)) (justify left))
     )
@@
       (effects (font (size 1.27 1.27)) (justify left))
     )
-    (property "Value" "10nF" (at 48.641 167.513 0)
+    (property "Value" "10n" (at 48.641 167.513 0)
       (effects (font (size 1.27 1.27)) (justify left))
     )
@@
       (effects (font (size 1.27 1.27)) (justify left))
     )
-    (property "Value" "100nF" (at 99.441 187.833 0)
+    (property "Value" "100n" (at 99.441 187.833 0)
       (effects (font (size 1.27 1.27)) (justify left))
     )
@@
       (effects (font (size 1.27 1.27)) (justify left))
     )
-    (property "Value" "100nF" (at 112.141 187.833 0)
+    (property "Value" "100n" (at 112.141 187.833 0)
       (effects (font (size 1.27 1.27)) (justify left))
     )
@@
       (effects (font (size 1.27 1.27)) (justify left))
     )
-    (property "Value" "100nF" (at 74.041 187.833 0)
+    (property "Value" "100n" (at 74.041 187.833 0)
       (effects (font (size 1.27 1.27)) (justify left))
     )
@@
       (effects (font (size 1.27 1.27)) (justify left))
     )
-    (property "Value" "100nF" (at 74.041 167.513 0)
+    (property "Value" "100n" (at 74.041 167.513 0)
       (effects (font (size 1.27 1.27)) (justify left))
     )
@@
       (effects (font (size 1.27 1.27)) (justify left))
     )
-    (property "Value" "100nF" (at 86.741 167.513 0)
+    (property "Value" "100n" (at 86.741 167.513 0)
       (effects (font (size 1.27 1.27)) (justify left))
     )
@@
       (effects (font (size 1.27 1.27)) (justify left))
     )
-    (property "Value" "100nF" (at 99.441 167.513 0)
+    (property "Value" "100n" (at 99.441 167.513 0)
       (effects (font (size 1.27 1.27)) (justify left))
     )
@@
       (effects (font (size 1.27 1.27)) (justify left))
     )
-    (property "Value" "100nF" (at 112.141 167.513 0)
+    (property "Value" "100n" (at 112.141 167.513 0)
       (effects (font (size 1.27 1.27)) (justify left))
     )
@@
       (effects (font (size 1.27 1.27)) (justify left))
     )
-    (property "Value" "100nF" (at 124.841 167.513 0)
+    (property "Value" "100n" (at 124.841 167.513 0)
       (effects (font (size 1.27 1.27)) (justify left))
     )
@@
       (effects (font (size 1.27 1.27)) (justify left))
     )
-    (property "Value" "100nF" (at 137.541 167.513 0)
+    (property "Value" "100n" (at 137.541 167.513 0)
       (effects (font (size 1.27 1.27)) (justify left))
     )
@@
       (effects (font (size 1.27 1.27)) (justify left))
     )
-    (property "Value" "100nF" (at 23.241 187.833 0)
+    (property "Value" "100n" (at 23.241 187.833 0)
       (effects (font (size 1.27 1.27)) (justify left))
     )
@@
       (effects (font (size 1.27 1.27)) (justify left))
     )
-    (property "Value" "100nF" (at 35.941 187.833 0)
+    (property "Value" "100n" (at 35.941 187.833 0)
       (effects (font (size 1.27 1.27)) (justify left))
     )
@@
       (effects (font (size 1.27 1.27)) (justify left))
     )
-    (property "Value" "100nF" (at 48.641 187.833 0)
+    (property "Value" "100n" (at 48.641 187.833 0)
       (effects (font (size 1.27 1.27)) (justify left))
     )
@@
       (effects (font (size 1.27 1.27)) (justify left))
     )
-    (property "Value" "100nF" (at 61.341 187.833 0)
+    (property "Value" "100n" (at 61.341 187.833 0)
       (effects (font (size 1.27 1.27)) (justify left))
     )
@@
       (effects (font (size 1.27 1.27)) (justify left))
     )
-    (property "Value" "100nF" (at 124.841 187.833 0)
+    (property "Value" "100n" (at 124.841 187.833 0)
       (effects (font (size 1.27 1.27)) (justify left))
     )
@@
       (effects (font (size 1.27 1.27)) (justify left))
     )
-    (property "Value" "100nF" (at 137.541 187.833 0)
+    (property "Value" "100n" (at 137.541 187.833 0)
       (effects (font (size 1.27 1.27)) (justify left))
     )
@@
       (effects (font (size 1.27 1.27)) (justify left))
     )
-    (property "Value" "100nF" (at 150.241 187.833 0)
+    (property "Value" "100n" (at 150.241 187.833 0)
       (effects (font (size 1.27 1.27)) (justify left))
     )
@@
       (effects (font (size 1.27 1.27)) (justify left))
     )
-    (property "Value" "100nF" (at 164.211 187.833 0)
-      (effects (font (size 1.27 1.27)) (justify left))
-    )
+    (property "Value" "100n" (at 164.211 187.833 0)
+      (effects (font (size 1.27 1.27)) (justify left))
+    )

Commit message: Tidy up switch symbols
Parts:
- SW1: value GameBoy_SW_SPDT -> SPDT; symbol Gekkio_Switch:GameBoy_SW_SPDT -> Gekkio_Switch:GameBoy_SW_SPDT_AGS
Changed lines of the file:
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@@
     )
   )
-  (symbol (lib_id "Gekkio_Switch:GameBoy_SW_SPDT") (at 80.01 45.72 0) (mirror y) (unit 1)
-    (in_bom yes) (on_board yes) (dnp no)
-    (property "Reference" "SW1" (at 80.01 38.5318 0)
+  (symbol (lib_id "Gekkio_Switch:GameBoy_SW_SPDT_AGS") (at 80.01 45.72 0) (mirror y) (unit 1)
+    (in_bom yes) (on_board yes) (dnp no) (fields_autoplaced)
+    (property "Reference" "SW1" (at 80.01 38.1 0)
       (effects (font (size 1.27 1.27)))
     )
-    (property "Value" "GameBoy_SW_SPDT" (at 80.01 40.8432 0)
+    (property "Value" "SPDT" (at 80.01 40.64 0)
       (effects (font (size 1.27 1.27)))
     )
