File: AGS-CPU-11/cartridge.kicad_sch (KiCad schematic)
At the start: 14 parts, among them P1 GameBoyAdvance_Cartridge_Moun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, SW13 GameBoy_SW_DPST

Commit message: Hide test point references
Parts:
- TP46, TP47, TP48, TP49, TP50: symbol Connector:TestPoint -> Connector:TestPoint_Small
Changed lines of the file:
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@@
   (junction (at 113.03 67.31) (diameter 0) (color 0 0 0 0)
   )
+  (junction (at 105.41 87.63) (diameter 0) (color 0 0 0 0)
+  )
   (junction (at 118.11 173.99) (diameter 0) (color 0 0 0 0)
   )
   (junction (at 85.09 41.91) (diameter 0) (color 0 0 0 0)
   )
-  (junction (at 105.41 87.63) (diameter 0) (color 0 0 0 0)
-  )
   (junction (at 82.55 161.29) (diameter 0) (color 0 0 0 0)
   )
+  (junction (at 76.2 161.29) (diameter 0) (color 0 0 0 0)
+  )
   (junction (at 96.52 46.99) (diameter 0) (color 0 0 0 0)
   )
-  (junction (at 76.2 161.29) (diameter 0) (color 0 0 0 0)
-  )
   (junction (at 113.03 46.99) (diameter 0) (color 0 0 0 0)
   )
@@
     (stroke (width 0) (type default) (color 0 0 0 0))
   )
+  (wire (pts (xy 105.41 85.09) (xy 105.41 87.63))
+    (stroke (width 0) (type default) (color 0 0 0 0))
+  )
   (wire (pts (xy 113.03 67.31) (xy 113.03 85.09))
     (stroke (width 0) (type default) (color 0 0 0 0))
@@
     (stroke (width 0) (type default) (color 0 0 0 0))
   )
-  (wire (pts (xy 82.55 161.29) (xy 76.2 161.29))
+  (wire (pts (xy 69.85 161.29) (xy 76.2 161.29))
     (stroke (width 0) (type default) (color 0 0 0 0))
   )
@@
     (stroke (width 0) (type default) (color 0 0 0 0))
   )
+  (wire (pts (xy 105.41 87.63) (xy 113.03 87.63))
+    (stroke (width 0) (type default) (color 0 0 0 0))
+  )
   (wire (pts (xy 107.95 158.75) (xy 107.95 161.29))
     (stroke (width 0) (type default) (color 0 0 0 0))
   )
   (wire (pts (xy 107.95 161.29) (xy 82.55 161.29))
+    (stroke (width 0) (type default) (color 0 0 0 0))
+  )
+  (wire (pts (xy 76.2 161.29) (xy 82.55 161.29))
     (stroke (width 0) (type default) (color 0 0 0 0))
   )
@@
     (stroke (width 0) (type default) (color 0 0 0 0))
   )
-  (wire (pts (xy 76.2 161.29) (xy 69.85 161.29))
-    (stroke (width 0) (type default) (color 0 0 0 0))
-  )
   (wire (pts (xy 113.03 44.45) (xy 113.03 46.99))
     (stroke (width 0) (type default) (color 0 0 0 0))
@@
     (stroke (width 0) (type default) (color 0 0 0 0))
   )
-  (wire (pts (xy 102.87 87.63) (xy 105.41 87.63))
-    (stroke (width 0) (type default) (color 0 0 0 0))
-  )
   (bus (pts (xy 105.41 102.87) (xy 105.41 105.41))
     (stroke (width 0) (type default) (color 0 0 0 0))
   )
   (bus (pts (xy 105.41 143.51) (xy 105.41 146.05))
+    (stroke (width 0) (type default) (color 0 0 0 0))
+  )
+  (wire (pts (xy 76.2 158.75) (xy 76.2 161.29))
     (stroke (width 0) (type default) (color 0 0 0 0))
   )
@@
     (stroke (width 0) (type default) (color 0 0 0 0))
   )
-  (wire (pts (xy 113.03 87.63) (xy 105.41 87.63))
+  (wire (pts (xy 102.87 87.63) (xy 105.41 87.63))
     (stroke (width 0) (type default) (color 0 0 0 0))
   )
@@
     (pin "1")
   )
-  (symbol (lib_id "Connector:TestPoint") (at 109.22 173.99 90) (unit 1)
-    (in_bom yes) (on_board yes)
-    (property "Reference" "TP50" (id 0) (at 107.3912 169.037 90))
-    (property "Value" "P1GND" (id 1) (at 107.3912 171.3484 90))
-    (property "Footprint" "" (id 2) (at 109.22 168.91 0)
-      (effects (font (size 1.27 1.27)) hide)
-    )
-    (property "Datasheet" "~" (id 3) (at 109.22 168.91 0)
+  (symbol (lib_id "Connector:TestPoint_Small") (at 109.22 173.99 180) (unit 1)
+    (in_bom yes) (on_board yes) (fields_autoplaced)
+    (property "Reference" "TP50" (id 0) (at 104.267 175.8188 90)
+      (effects (font (size 1.27 1.27)) hide)
+    )
+    (property "Value" "P1GND" (id 1) (at 107.95 173.9899 0)
+      (effects (font (size 1.27 1.27)) (justify left))
+    )
+    (property "Footprint" "" (id 2) (at 104.14 173.99 0)
+      (effects (font (size 1.27 1.27)) hide)
+    )
+    (property "Datasheet" "~" (id 3) (at 104.14 173.99 0)
       (effects (font (size 1.27 1.27)) hide)
     )
@@
     (pin "2")
   )
-  (symbol (lib_id "Connector:TestPoint") (at 105.41 87.63 0) (unit 1)
-    (in_bom yes) (on_board yes)
-    (property "Reference" "TP49" (id 0) (at 105.41 79.375 0))
-    (property "Value" "PHI" (id 1) (at 105.41 81.6864 0))
-    (property "Footprint" "" (id 2) (at 110.49 87.63 0)
-      (effects (font (size 1.27 1.27)) hide)
-    )
-    (property "Datasheet" "~" (id 3) (at 110.49 87.63 0)
+  (symbol (lib_id "Connector:TestPoint_Small") (at 105.41 85.09 90) (unit 1)
+    (in_bom yes) (on_board yes) (fields_autoplaced)
+    (property "Reference" "TP49" (id 0) (at 97.155 85.09 0)
+      (effects (font (size 1.27 1.27)) hide)
+    )
+    (property "Value" "PHI" (id 1) (at 105.41 82.55 90))
+    (property "Footprint" "" (id 2) (at 105.41 80.01 0)
+      (effects (font (size 1.27 1.27)) hide)
+    )
+    (property "Datasheet" "~" (id 3) (at 105.41 80.01 0)
       (effects (font (size 1.27 1.27)) hide)
     )
@@
     (pin "2")
   )
-  (symbol (lib_id "Connector:TestPoint") (at 76.2 161.29 0) (unit 1)
-    (in_bom yes) (on_board yes)
-    (property "Reference" "TP46" (id 0) (at 76.2 153.035 0))
-    (property "Value" "RES" (id 1) (at 76.2 155.3464 0))
-    (property "Footprint" "" (id 2) (at 81.28 161.29 0)
-      (effects (font (size 1.27 1.27)) hide)
-    )
-    (property "Datasheet" "~" (id 3) (at 81.28 161.29 0)
+  (symbol (lib_id "Connector:TestPoint_Small") (at 76.2 158.75 90) (unit 1)
+    (in_bom yes) (on_board yes) (fields_autoplaced)
+    (property "Reference" "TP46" (id 0) (at 67.945 158.75 0)
+      (effects (font (size 1.27 1.27)) hide)
+    )
+    (property "Value" "RES" (id 1) (at 76.2 156.21 90))
+    (property "Footprint" "" (id 2) (at 76.2 153.67 0)
+      (effects (font (size 1.27 1.27)) hide)
+    )
+    (property "Datasheet" "~" (id 3) (at 76.2 153.67 0)
       (effects (font (size 1.27 1.27)) hide)
     )
@@
     (pin "2")
   )
-  (symbol (lib_id "Connector:TestPoint") (at 85.09 38.1 0) (unit 1)
-    (in_bom yes) (on_board yes)
-    (property "Reference" "TP47" (id 0) (at 86.5632 35.1028 0)
-      (effects (font (size 1.27 1.27)) (justify left))
-    )
-    (property "Value" "IN35" (id 1) (at 86.5632 37.4142 0)
-      (effects (font (size 1.27 1.27)) (justify left))
-    )
-    (property "Footprint" "" (id 2) (at 90.17 38.1 0)
-      (effects (font (size 1.27 1.27)) hide)
-    )
-    (property "Datasheet" "~" (id 3) (at 90.17 38.1 0)
+  (symbol (lib_id "Connector:TestPoint_Small") (at 85.09 38.1 90) (unit 1)
+    (in_bom yes) (on_board yes) (fields_autoplaced)
+    (property "Reference" "TP47" (id 0) (at 82.0928 36.6268 0)
+      (effects (font (size 1.27 1.27)) (justify left) hide)
+    )
+    (property "Value" "IN35" (id 1) (at 85.09 35.56 90))
+    (property "Footprint" "" (id 2) (at 85.09 33.02 0)
+      (effects (font (size 1.27 1.27)) hide)
+    )
+    (property "Datasheet" "~" (id 3) (at 85.09 33.02 0)
       (effects (font (size 1.27 1.27)) hide)
     )
@@
     (pin "1")
   )
-  (symbol (lib_id "Connector:TestPoint") (at 96.52 38.1 0) (unit 1)
-    (in_bom yes) (on_board yes)
-    (property "Reference" "TP48" (id 0) (at 97.9932 35.1028 0)
-      (effects (font (size 1.27 1.27)) (justify left))
-    )
-    (property "Value" "VDD35" (id 1) (at 97.9932 37.4142 0)
-      (effects (font (size 1.27 1.27)) (justify left))
-    )
-    (property "Footprint" "" (id 2) (at 101.6 38.1 0)
-      (effects (font (size 1.27 1.27)) hide)
-    )
-    (property "Datasheet" "~" (id 3) (at 101.6 38.1 0)
-      (effects (font (size 1.27 1.27)) hide)
-    )
+  (symbol (lib_id "Connector:TestPoint_Small") (at 96.52 38.1 90) (unit 1)
+    (in_bom yes) (on_board yes) (fields_autoplaced)
+    (property "Reference" "TP48" (id 0) (at 93.5228 36.6268 0)
+      (effects (font (size 1.27 1.27)) (justify left) hide)
+    )
+    (property "Value" "VDD35" (id 1) (at 96.52 35.56 90))
+    (property "Footprint" "" (id 2) (at 96.52 33.02 0)
+      (effects (font (size 1.27 1.27)) hide)
+    )
+    (property "Datasheet" "~" (id 3) (at 96.52 33.02 0)
+      (effects (font (size 1.27 1.27)) hide)
+    )

Commit message: Release: AGB-CPU-11 rev D
Other:
- title: AGS-CPU-11 - Cartridge slot -> AGS-CPU-11
Changed lines of the file:
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@@
   (paper "A4")
   (title_block
-    (title "AGS-CPU-11 - Cartridge slot")
-    (date "2021-07-26")
-    (rev "C")
+    (title "AGS-CPU-11")
+    (date "2022-01-02")
+    (rev "D")
     (company "https://gekkio.fi")
     (comment 1 "https://github.com/Gekkio/gb-schematics")

Commit message: Remove Farad/Henry units
Parts:
- C3: value 100nF -> 100n
Changed lines of the file:
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@@
       (effects (font (size 1.27 1.27)) (justify left))
     )
-    (property "Value" "100nF" (at 123.571 72.263 0)
+    (property "Value" "100n" (at 123.571 72.263 0)
       (effects (font (size 1.27 1.27)) (justify left))
     )

Commit message: Tidy up switch symbols
Parts:
- SW13: value GameBoy_SW_DPST -> DPDT; symbol Gekkio_Switch:GameBoy_SW_DPST -> Gekkio_Switch:GameBoy_SW_DPDT_AGS
Changed lines of the file:
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@@
     )
   )
-  (symbol (lib_id "Gekkio_Switch:GameBoy_SW_DPST") (at 71.12 44.45 0) (mirror y) (unit 1)
-    (in_bom yes) (on_board yes) (dnp no)
-    (property "Reference" "SW13" (at 71.12 35.179 0)
+  (symbol (lib_id "Gekkio_Switch:GameBoy_SW_DPDT_AGS") (at 71.12 44.45 0) (mirror y) (unit 1)
+    (in_bom yes) (on_board yes) (dnp no) (fields_autoplaced)
+    (property "Reference" "SW13" (at 71.12 34.29 0)
       (effects (font (size 1.27 1.27)))
     )
-    (property "Value" "GameBoy_SW_DPST" (at 71.12 37.4904 0)
+    (property "Value" "DPDT" (at 71.12 36.83 0)
       (effects (font (size 1.27 1.27)))
     )
