File: DC-CONV-DMG-AB/DC-CONV-DMG-AB.kicad_sch (KiCad schematic)
At the start: 19 parts, among them J1 Conn_01x04, Q1 2SD1664R, Q2 2SD1328, T1 GameBoy_Transformer_DMG

Commit message: Release: DC-CONV-DMG-AB rev B
Parts:
- D2: value D_Schottky -> 1SS294; footprint (none) -> Package_TO_SOT_SMD:SOT-23; symbol Device:D_Schottky -> Gekkio_Diode:1SS294
- T1: value GameBoy_Transformer_DMG -> 223 or 231
Connections:
- net VOUT+: now also D2.3 (K); no longer D2.1 (K)
- net at T1.6: now also D2.1 (A); no longer D2.2 (A)
Other:
- moved on the sheet: Q2
Changed lines of the file:
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@@
   (title_block
     (title "DC-CONV-DMG-A / DC-CONV-DMG-B")
-    (date "2022-01-02")
-    (rev "A")
+    (date "2022-01-12")
+    (rev "B")
     (company "https://gekkio.fi")
     (comment 1 "https://github.com/gekkio/gb-schematics")
@@
     (stroke (width 0) (type default) (color 0 0 0 0))
   )
-  (wire (pts (xy 81.28 148.59) (xy 85.09 148.59))
-    (stroke (width 0) (type default) (color 0 0 0 0))
-  )
   (wire (pts (xy 152.4 69.85) (xy 179.07 69.85))
     (stroke (width 0) (type default) (color 0 0 0 0))
@@
     (stroke (width 0) (type default) (color 0 0 0 0))
   )
-  (wire (pts (xy 81.28 158.75) (xy 85.09 158.75))
-    (stroke (width 0) (type default) (color 0 0 0 0))
-  )
   (polyline (pts (xy 67.31 95.25) (xy 67.31 113.03))
     (stroke (width 0.3) (type default) (color 0 0 0 0))
@@
     (stroke (width 0) (type default) (color 0 0 0 0))
   )
-  (wire (pts (xy 92.71 153.67) (xy 97.79 153.67))
+  (wire (pts (xy 88.9 153.67) (xy 97.79 153.67))
     (stroke (width 0) (type default) (color 0 0 0 0))
   )
@@
     (in_bom yes) (on_board yes) (fields_autoplaced)
     (property "Reference" "T1" (id 0) (at 123.19 59.69 0))
-    (property "Value" "GameBoy_Transformer_DMG" (id 1) (at 123.19 62.23 0))
+    (property "Value" "223 or 231" (id 1) (at 123.19 62.23 0))
     (property "Footprint" "Gekkio_Transformer_THT:Transformer_GameBoy_DMG" (id 2) (at 123.19 90.17 0)
       (effects (font (size 1.27 1.27)) hide)
@@
     (pin "1")
   )
-  (symbol (lib_id "Device:D_Schottky") (at 147.32 69.85 0) (mirror y) (unit 1)
-    (in_bom yes) (on_board yes) (fields_autoplaced)
-    (property "Reference" "D2" (id 0) (at 147.6375 63.5 0))
-    (property "Value" "D_Schottky" (id 1) (at 147.6375 66.04 0))
-    (property "Footprint" "" (id 2) (at 147.32 69.85 0)
-      (effects (font (size 1.27 1.27)) hide)
-    )
-    (property "Datasheet" "~" (id 3) (at 147.32 69.85 0)
-      (effects (font (size 1.27 1.27)) hide)
-    )
-    (pin "1")
-    (pin "2")
+  (symbol (lib_id "Gekkio_Diode:1SS294") (at 147.32 69.85 0) (mirror y) (unit 1)
+    (in_bom yes) (on_board yes) (fields_autoplaced)
+    (property "Reference" "D2" (id 0) (at 147.6375 62.23 0))
+    (property "Value" "1SS294" (id 1) (at 147.6375 64.77 0))
+    (property "Footprint" "Package_TO_SOT_SMD:SOT-23" (id 2) (at 147.32 74.295 0)
+      (effects (font (size 1.27 1.27)) hide)
+    )
+    (property "Datasheet" "https://toshiba.semicon-storage.com/info/docget.jsp?did=3290&prodName=1SS294" (id 3) (at 147.32 76.2 0)
+      (effects (font (size 1.27 1.27)) hide)
+    )
+    (pin "1")
+    (pin "2")
+    (pin "3")
   )
   (symbol (lib_id "Device:D") (at 147.32 97.79 0) (unit 1)
@@
     (pin "2")
   )
-  (symbol (lib_id "Device:Q_NPN_BEC") (at 87.63 153.67 0) (mirror y) (unit 1)
-    (in_bom yes) (on_board yes)
+  (symbol (lib_id "Device:Q_NPN_BEC") (at 83.82 153.67 0) (mirror y) (unit 1)
+    (in_bom yes) (on_board yes) (fields_autoplaced)
     (property "Reference" "Q2" (id 0) (at 78.74 152.3999 0)
       (effects (font (size 1.27 1.27)) (justify left))
@@
       (effects (font (size 1.27 1.27)) (justify left))
     )
-    (property "Footprint" "" (id 2) (at 82.55 151.13 0)
-      (effects (font (size 1.27 1.27)) hide)
-    )
-    (property "Datasheet" "~" (id 3) (at 87.63 153.67 0)
+    (property "Footprint" "" (id 2) (at 78.74 151.13 0)
+      (effects (font (size 1.27 1.27)) hide)
+    )
+    (property "Datasheet" "~" (id 3) (at 83.82 153.67 0)
       (effects (font (size 1.27 1.27)) hide)
     )
@@
     )
     (path "/00000000-0000-0000-0000-00005f093dd4"
-      (reference "D2") (unit 1) (value "D_Schottky") (footprint "")
+      (reference "D2") (unit 1) (value "1SS294") (footprint "Package_TO_SOT_SMD:SOT-23")
     )
     (path "/00000000-0000-0000-0000-00005f0bd48e"
@@
     )
     (path "/00000000-0000-0000-0000-00005f059b3c"
-      (reference "T1") (unit 1) (value "GameBoy_Transformer_DMG") (footprint "Gekkio_Transformer_THT:Transformer_GameBoy_DMG")
-    )
-  )
+      (reference "T1") (unit 1) (value "223 or 231") (footprint "Gekkio_Transformer_THT:Transformer_GameBoy_DMG")
+    )
+  )

Commit message: Remove Farad/Henry units
Parts:
- C1: value 680nF -> 680n
- C2: value 1nF -> 1n
- C3: value 8.2nF -> 8.2n
- C4: value 33uF -> 33u
- C5: value 10uF -> 10u
- L1: value 1uH -> 1u
Changed lines of the file:
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@@
       (effects (font (size 1.27 1.27)))
     )
-    (property "Value" "1uH" (at 31.75 60.96 90)
+    (property "Value" "1u" (at 31.75 60.96 90)
       (effects (font (size 1.27 1.27)))
     )
@@
       (effects (font (size 1.27 1.27)))
     )
-    (property "Value" "1nF" (at 101.6 101.6 90)
+    (property "Value" "1n" (at 101.6 101.6 90)
       (effects (font (size 1.27 1.27)))
     )
@@
       (effects (font (size 1.27 1.27)) (justify left))
     )
-    (property "Value" "680nF" (at 41.91 72.3899 0)
+    (property "Value" "680n" (at 41.91 72.3899 0)
       (effects (font (size 1.27 1.27)) (justify left))
     )
@@
       (effects (font (size 1.27 1.27)) (justify left))
     )
-    (property "Value" "10uF" (at 182.88 75.3109 0)
+    (property "Value" "10u" (at 182.88 75.3109 0)
       (effects (font (size 1.27 1.27)) (justify left))
     )
@@
       (effects (font (size 1.27 1.27)) (justify left))
     )
-    (property "Value" "33uF" (at 182.88 90.5509 0)
+    (property "Value" "33u" (at 182.88 90.5509 0)
       (effects (font (size 1.27 1.27)) (justify left))
     )
@@
       (effects (font (size 1.27 1.27)) (justify left))
     )
-    (property "Value" "8.2nF" (at 119.38 161.2899 0)
-      (effects (font (size 1.27 1.27)) (justify left))
-    )
+    (property "Value" "8.2n" (at 119.38 161.2899 0)
+      (effects (font (size 1.27 1.27)) (justify left))
+    )
