File: DC-CONV-DMG-C/DC-CONV-DMG-C.kicad_sch (KiCad schematic)
At the start: 18 parts, among them J1 Conn_01x04, Q1 2SD1664R, Q2 2SC2412, T1 280

Commit message: Remove Farad/Henry units
Parts:
- C1: value 470nF -> 470n
- C2: value 680pF -> 680p
- C3: value 8.2nF -> 8.2n
- C4: value 33uF -> 33u
- C5: value 100uF -> 100u
Changed lines of the file:
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@@
       (effects (font (size 1.27 1.27)))
     )
-    (property "Value" "680pF" (at 101.6 101.6 90)
+    (property "Value" "680p" (at 101.6 101.6 90)
       (effects (font (size 1.27 1.27)))
     )
@@
       (effects (font (size 1.27 1.27)) (justify left))
     )
-    (property "Value" "470nF" (at 40.64 72.3899 0)
+    (property "Value" "470n" (at 40.64 72.3899 0)
       (effects (font (size 1.27 1.27)) (justify left))
     )
@@
       (effects (font (size 1.27 1.27)) (justify left))
     )
-    (property "Value" "100uF" (at 182.88 75.3109 0)
+    (property "Value" "100u" (at 182.88 75.3109 0)
       (effects (font (size 1.27 1.27)) (justify left))
     )
@@
       (effects (font (size 1.27 1.27)) (justify left))
     )
-    (property "Value" "33uF" (at 182.88 90.5509 0)
+    (property "Value" "33u" (at 182.88 90.5509 0)
       (effects (font (size 1.27 1.27)) (justify left))
     )
@@
       (effects (font (size 1.27 1.27)) (justify left))
     )
-    (property "Value" "8.2nF" (at 119.38 161.2899 0)
-      (effects (font (size 1.27 1.27)) (justify left))
-    )
+    (property "Value" "8.2n" (at 119.38 161.2899 0)
+      (effects (font (size 1.27 1.27)) (justify left))
+    )
