File: LSEP01088A1/LSEP01088A1.kicad_sch (KiCad schematic)
At the start: 31 parts, among them J1 Conn_02x03_Counter_Clockwise, Q1 2SD601A, Q2 2SD601A, Q3 2SD601A, Q4 2SD1119, Q5 2SD601A, T1 066

Commit message: Remove Farad/Henry units
Parts:
- C1: value 4.7uF -> 4.7u
- C2, C5: value 1.5uF -> 1.5u
- C3, C6, C8: value 100nF -> 100n
- C4: value 1nF -> 1n
- C7: value 22nF -> 22n
- C9: value 150pF -> 150p
Changed lines of the file:
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@@
       (effects (font (size 1.27 1.27)) (justify left))
     )
-    (property "Value" "1nF" (at 144.78 76.1999 0)
+    (property "Value" "1n" (at 144.78 76.1999 0)
       (effects (font (size 1.27 1.27)) (justify left))
     )
@@
       (effects (font (size 1.27 1.27)) (justify right))
     )
-    (property "Value" "150pF" (at 140.97 123.1899 0)
+    (property "Value" "150p" (at 140.97 123.1899 0)
       (effects (font (size 1.27 1.27)) (justify right))
     )
@@
       (effects (font (size 1.27 1.27)) (justify left))
     )
-    (property "Value" "100nF" (at 210.82 77.4699 0)
+    (property "Value" "100n" (at 210.82 77.4699 0)
       (effects (font (size 1.27 1.27)) (justify left))
     )
@@
       (effects (font (size 1.27 1.27)) (justify right))
     )
-    (property "Value" "1.5uF" (at 58.42 88.8999 0)
+    (property "Value" "1.5u" (at 58.42 88.8999 0)
       (effects (font (size 1.27 1.27)) (justify right))
     )
@@
       (effects (font (size 1.27 1.27)))
     )
-    (property "Value" "100nF" (at 130.81 97.79 90)
+    (property "Value" "100n" (at 130.81 97.79 90)
       (effects (font (size 1.27 1.27)))
     )
@@
       (effects (font (size 1.27 1.27)) (justify left))
     )
-    (property "Value" "1.5uF" (at 210.82 60.9599 0)
+    (property "Value" "1.5u" (at 210.82 60.9599 0)
       (effects (font (size 1.27 1.27)) (justify left))
     )
@@
       (effects (font (size 1.27 1.27)) (justify right))
     )
-    (property "Value" "22nF" (at 134.62 144.7799 0)
+    (property "Value" "22n" (at 134.62 144.7799 0)
       (effects (font (size 1.27 1.27)) (justify right))
     )
@@
       (effects (font (size 1.27 1.27)) (justify left))
     )
-    (property "Value" "4.7uF" (at 29.21 67.3099 0)
+    (property "Value" "4.7u" (at 29.21 67.3099 0)
       (effects (font (size 1.27 1.27)) (justify left))
     )
@@
       (effects (font (size 1.27 1.27)))
     )
-    (property "Value" "100nF" (at 158.75 88.9 90)
-      (effects (font (size 1.27 1.27)))
-    )
+    (property "Value" "100n" (at 158.75 88.9 90)
+      (effects (font (size 1.27 1.27)))
+    )
