File: MGB-DCDC-B/MGB-DCDC-B.kicad_sch (KiCad schematic)
At the start: 29 parts, among them J1 Conn_02x03_Counter_Clockwise, Q1 KTC3875S, Q2 KTC3875S, Q3 KTC3875S, Q4 2SD2150, Q5 KTC3875S, T1 015

Commit message: Remove Farad/Henry units
Parts:
- C1: value 2.2uF -> 2.2u
- C2, C5: value 1uF -> 1u
- C3, C6: value 100nF -> 100n
- C4: value 510pF -> 510p
- C7: value 33nF -> 33n
- C8: value 100pF -> 100p
- C9: value 51pF -> 51p
Changed lines of the file:
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@@
       (effects (font (size 1.27 1.27)) (justify left))
     )
-    (property "Value" "510pF" (at 144.78 76.1999 0)
+    (property "Value" "510p" (at 144.78 76.1999 0)
       (effects (font (size 1.27 1.27)) (justify left))
     )
@@
       (effects (font (size 1.27 1.27)) (justify right))
     )
-    (property "Value" "51pF" (at 140.97 123.1899 0)
+    (property "Value" "51p" (at 140.97 123.1899 0)
       (effects (font (size 1.27 1.27)) (justify right))
     )
@@
       (effects (font (size 1.27 1.27)) (justify left))
     )
-    (property "Value" "100nF" (at 210.82 77.4699 0)
+    (property "Value" "100n" (at 210.82 77.4699 0)
       (effects (font (size 1.27 1.27)) (justify left))
     )
@@
       (effects (font (size 1.27 1.27)) (justify right))
     )
-    (property "Value" "1uF" (at 58.42 88.8999 0)
+    (property "Value" "1u" (at 58.42 88.8999 0)
       (effects (font (size 1.27 1.27)) (justify right))
     )
@@
       (effects (font (size 1.27 1.27)))
     )
-    (property "Value" "100nF" (at 130.81 97.79 90)
+    (property "Value" "100n" (at 130.81 97.79 90)
       (effects (font (size 1.27 1.27)))
     )
@@
       (effects (font (size 1.27 1.27)) (justify left))
     )
-    (property "Value" "1uF" (at 210.82 60.9599 0)
+    (property "Value" "1u" (at 210.82 60.9599 0)
       (effects (font (size 1.27 1.27)) (justify left))
     )
@@
       (effects (font (size 1.27 1.27)) (justify right))
     )
-    (property "Value" "33nF" (at 134.62 148.5899 0)
+    (property "Value" "33n" (at 134.62 148.5899 0)
       (effects (font (size 1.27 1.27)) (justify right))
     )
@@
       (effects (font (size 1.27 1.27)))
     )
-    (property "Value" "100pF" (at 114.3 109.22 90)
+    (property "Value" "100p" (at 114.3 109.22 90)
       (effects (font (size 1.27 1.27)))
     )
@@
       (effects (font (size 1.27 1.27)) (justify left))
     )
-    (property "Value" "2.2uF" (at 29.21 67.3099 0)
-      (effects (font (size 1.27 1.27)) (justify left))
-    )
+    (property "Value" "2.2u" (at 29.21 67.3099 0)
+      (effects (font (size 1.27 1.27)) (justify left))
+    )
