File: MGL-CPU-01/MGL-CPU-01.kicad_sch (KiCad schematic)
At the start: 53 parts, among them P1 GameBoy_Cartridge, U1 CPU MGB, U2 LH5164AN-10L, U6 PST9135N, X1 4.194304 MHz

Commit message: Remove Farad/Henry units
Parts:
- C1, C2: value 27pF -> 27p
- C10, C11, C12: value 15nF -> 15n
- C17: value 150nF -> 150n
Changed lines of the file:
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@@
       (effects (font (size 1.27 1.27)) (justify left))
     )
-    (property "Value" "15nF" (at 272.161 154.813 0)
+    (property "Value" "15n" (at 272.161 154.813 0)
       (effects (font (size 1.27 1.27)) (justify left))
     )
@@
       (effects (font (size 1.27 1.27)) (justify left))
     )
-    (property "Value" "15nF" (at 230.251 154.813 0)
+    (property "Value" "15n" (at 230.251 154.813 0)
       (effects (font (size 1.27 1.27)) (justify left))
     )
@@
       (effects (font (size 1.27 1.27)) (justify left))
     )
-    (property "Value" "27pF" (at 28.321 114.173 0)
+    (property "Value" "27p" (at 28.321 114.173 0)
       (effects (font (size 1.27 1.27)) (justify left))
     )
@@
       (effects (font (size 1.27 1.27)) (justify left))
     )
-    (property "Value" "27pF" (at 41.021 114.173 0)
+    (property "Value" "27p" (at 41.021 114.173 0)
       (effects (font (size 1.27 1.27)) (justify left))
     )
@@
       (effects (font (size 1.27 1.27)) (justify left))
     )
-    (property "Value" "150nF" (at 43.561 69.723 0)
+    (property "Value" "150n" (at 43.561 69.723 0)
       (effects (font (size 1.27 1.27)) (justify left))
     )
@@
       (effects (font (size 1.27 1.27)) (justify left))
     )
-    (property "Value" "15nF" (at 112.141 167.513 0)
-      (effects (font (size 1.27 1.27)) (justify left))
-    )
+    (property "Value" "15n" (at 112.141 167.513 0)
+      (effects (font (size 1.27 1.27)) (justify left))
+    )
