File: MGL-CPU-01/power.kicad_sch (KiCad schematic)
At the start: 44 parts, among them J1 EL, P4 DC 3V, Q2 2SC4081, Q3 2SD1781K, Q4 2SD1781K, T1 GameBoy_Transformer_MGL_EL, U5 DC/DC

Commit message: Update to latest KiCad
Parts:
- SW1: value (none) -> DP3T

Commit message: Remove Farad/Henry units
Parts:
- C29: value 1uF -> 1u
- C30, C32: value 330uF -> 330u
- C33: value 6.8uF -> 6.8u
- C34: value 220nF -> 220n
- C36: value 10nF -> 10n
- C38: value 33uF -> 33u
- C39: value 15nF -> 15n
Changed lines of the file:
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@@
       (effects (font (size 1.27 1.27)) (justify left))
     )
-    (property "Value" "330uF" (at 64.77 101.9809 0)
+    (property "Value" "330u" (at 64.77 101.9809 0)
       (effects (font (size 1.27 1.27)) (justify left))
     )
@@
       (effects (font (size 1.27 1.27)) (justify left))
     )
-    (property "Value" "6.8uF" (at 99.441 102.743 0)
+    (property "Value" "6.8u" (at 99.441 102.743 0)
       (effects (font (size 1.27 1.27)) (justify left))
     )
@@
       (effects (font (size 1.27 1.27)) (justify right))
     )
-    (property "Value" "1uF" (at 100.33 115.9509 0)
+    (property "Value" "1u" (at 100.33 115.9509 0)
       (effects (font (size 1.27 1.27)) (justify right))
     )
@@
       (effects (font (size 1.27 1.27)) (justify right))
     )
-    (property "Value" "330uF" (at 48.26 101.9809 0)
+    (property "Value" "330u" (at 48.26 101.9809 0)
       (effects (font (size 1.27 1.27)) (justify right))
     )
@@
       (effects (font (size 1.27 1.27)))
     )
-    (property "Value" "10nF" (at 226.06 120.65 90)
+    (property "Value" "10n" (at 226.06 120.65 90)
       (effects (font (size 1.27 1.27)))
     )
@@
       (effects (font (size 1.27 1.27)) (justify left))
     )
-    (property "Value" "15nF" (at 107.95 58.4199 0)
+    (property "Value" "15n" (at 107.95 58.4199 0)
       (effects (font (size 1.27 1.27)) (justify left))
     )
@@
       (effects (font (size 1.27 1.27)) (justify left))
     )
-    (property "Value" "33uF" (at 214.63 94.3609 0)
+    (property "Value" "33u" (at 214.63 94.3609 0)
       (effects (font (size 1.27 1.27)) (justify left))
     )
@@
       (effects (font (size 1.27 1.27)) (justify left))
     )
-    (property "Value" "220nF" (at 201.93 118.1099 0)
-      (effects (font (size 1.27 1.27)) (justify left))
-    )
+    (property "Value" "220n" (at 201.93 118.1099 0)
+      (effects (font (size 1.27 1.27)) (justify left))
+    )

Commit message: Add some power-related information
Other:
- note added: "Main power inputs (DC jack, battery) 0.7W"
- note added: "Plug: 2.35 mm x 0.75 mm Center positive polarity"
- note removed: "Main power inputs (DC jack, battery)"
Changed lines of the file:
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@@
     (effects (font (size 1.27 1.27)) (justify left bottom))
+  )
+  (text "Plug: 2.35 mm x 0.75 mm\nCenter positive polarity" (at 39.37 55.88 0)
+    (effects (font (size 1.27 1.27)) (justify right bottom))
   )
   (text "*see Note 3" (at 158.75 66.04 0)
     (effects (font (size 1.27 1.27)) (justify right bottom))
   )
-  (text "Main power inputs (DC jack, battery)" (at 134.62 26.67 0)
+  (text "Main power inputs (DC jack, battery)\n0.7W" (at 134.62 29.21 0)
     (effects (font (size 1.27 1.27) (thickness 0.254) bold) (justify right bottom))
   )

Commit message: Tidy up switch symbols
Parts:
- SW1: symbol MGL-CPU-01:GameBoy_SW_MGL -> Gekkio_Switch:GameBoy_SW_DP3T_MGL
Changed lines of the file:
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@@
     )
   )
-  (symbol (lib_id "MGL-CPU-01:GameBoy_SW_MGL") (at 172.72 53.34 0) (mirror y) (unit 1)
+  (symbol (lib_id "Gekkio_Switch:GameBoy_SW_DP3T_MGL") (at 172.72 53.34 0) (mirror y) (unit 1)
     (in_bom yes) (on_board yes) (dnp no) (fields_autoplaced)
     (property "Reference" "SW1" (at 172.4279 41.91 0)
