File: MGL-CPU-01/lcd.kicad_sch (KiCad schematic)
At the start: 34 parts, among them P2 LCD FPC, Q1 2SA1576A, U4 IR3E02

Commit message: Remove Farad/Henry units
Parts:
- C20, C21, C23: value 1.5uF -> 1.5u
- C22, C24: value 1uF -> 1u
- C28: value 10uF -> 10u
- C3: value 47pF -> 47p
Changed lines of the file:
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@@
       (effects (font (size 1.27 1.27)) (justify left))
     )
-    (property "Value" "10uF" (at 49.911 63.373 0)
+    (property "Value" "10u" (at 49.911 63.373 0)
       (effects (font (size 1.27 1.27)) (justify left))
     )
@@
       (effects (font (size 1.27 1.27)) (justify left))
     )
-    (property "Value" "47pF" (at 115.951 60.833 0)
+    (property "Value" "47p" (at 115.951 60.833 0)
       (effects (font (size 1.27 1.27)) (justify left))
     )
@@
       (effects (font (size 1.27 1.27)) (justify left))
     )
-    (property "Value" "1uF" (at 187.071 58.293 0)
+    (property "Value" "1u" (at 187.071 58.293 0)
       (effects (font (size 1.27 1.27)) (justify left))
     )
@@
       (effects (font (size 1.27 1.27)) (justify left))
     )
-    (property "Value" "1uF" (at 165.481 58.293 0)
+    (property "Value" "1u" (at 165.481 58.293 0)
       (effects (font (size 1.27 1.27)) (justify left))
     )
@@
       (effects (font (size 1.27 1.27)) (justify left))
     )
-    (property "Value" "1.5uF" (at 142.621 58.293 0)
+    (property "Value" "1.5u" (at 142.621 58.293 0)
       (effects (font (size 1.27 1.27)) (justify left))
     )
@@
       (effects (font (size 1.27 1.27)) (justify left))
     )
-    (property "Value" "1.5uF" (at 154.051 58.293 0)
+    (property "Value" "1.5u" (at 154.051 58.293 0)
       (effects (font (size 1.27 1.27)) (justify left))
     )
@@
       (effects (font (size 1.27 1.27)) (justify left))
     )
-    (property "Value" "1.5uF" (at 175.641 58.293 0)
-      (effects (font (size 1.27 1.27)) (justify left))
-    )
+    (property "Value" "1.5u" (at 175.641 58.293 0)
+      (effects (font (size 1.27 1.27)) (justify left))
+    )

Commit message: Tidy up potentiometer symbols, add contrast pot symbols
Parts:
- removed VR2: 30k, symbol Device:R_Variable
- added VR2: 30k, symbol Gekkio_Device_Specialized:R_Potentiometer_GameBoy_Contrast_MGB
Connections:
- net GND: now also VR2.MP (MountPin)
- net VR: now also VR2.1 (4), VR2.2
- net at JP1.1 (A), TP64.1: now also VR2.5
Other:
- note removed: "TODO: more specific symbol"
- moved on the sheet: C20, C21, C22, C23, C24, C3, Q1, R1, U4
