File: MGL-CPU-01/link_port.kicad_sch (KiCad schematic)
At the start: 9 parts, among them P3 GameBoy_LinkPort

Commit message: Remove Farad/Henry units
Parts:
- C4, C5, C6, C7: value 100pF -> 100p
- C9: value 15nF -> 15n
Changed lines of the file:
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@@
       (effects (font (size 1.27 1.27)) (justify left))
     )
-    (property "Value" "15nF" (at 216.281 120.523 0)
+    (property "Value" "15n" (at 216.281 120.523 0)
       (effects (font (size 1.27 1.27)) (justify left))
     )
@@
       (effects (font (size 1.27 1.27)) (justify left))
     )
-    (property "Value" "100pF" (at 198.501 120.523 0)
+    (property "Value" "100p" (at 198.501 120.523 0)
       (effects (font (size 1.27 1.27)) (justify left))
     )
@@
       (effects (font (size 1.27 1.27)) (justify left))
     )
-    (property "Value" "100pF" (at 185.801 120.523 0)
+    (property "Value" "100p" (at 185.801 120.523 0)
       (effects (font (size 1.27 1.27)) (justify left))
     )
@@
       (effects (font (size 1.27 1.27)) (justify left))
     )
-    (property "Value" "100pF" (at 173.101 120.523 0)
+    (property "Value" "100p" (at 173.101 120.523 0)
       (effects (font (size 1.27 1.27)) (justify left))
     )
@@
       (effects (font (size 1.27 1.27)) (justify left))
     )
-    (property "Value" "100pF" (at 160.401 120.523 0)
+    (property "Value" "100p" (at 160.401 120.523 0)
       (effects (font (size 1.27 1.27)) (justify left))
     )
