File: DMG-CPU-06/power.kicad_sch (KiCad schematic)
At the start: 8 parts, among them J1 Conn_01x04, SW1 DPST

Commit message: Tidy up switch symbols
Parts:
- SW1: value DPST -> DPDT; symbol Gekkio_Switch:GameBoy_SW_DMG -> Gekkio_Switch:GameBoy_SW_DPDT_DMG
Changed lines of the file:
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@@
     )
   )
-  (symbol (lib_id "Gekkio_Switch:GameBoy_SW_DMG") (at 165.1 64.77 0) (unit 1)
+  (symbol (lib_id "Gekkio_Switch:GameBoy_SW_DPDT_DMG") (at 165.1 64.77 0) (unit 1)
     (in_bom yes) (on_board yes) (dnp no) (fields_autoplaced)
     (property "Reference" "SW1" (at 165.1 54.61 0)
       (effects (font (size 1.27 1.27)))
     )
-    (property "Value" "DPST" (at 165.1 57.15 0)
+    (property "Value" "DPDT" (at 165.1 57.15 0)
       (effects (font (size 1.27 1.27)))
     )
